File: KiCad/Daikin.kicad_pcb (KiCad board)
At the start: 2 copper layers, 13.2 x 19.5 mm, 19 parts, among them J1 SPOX, J2 Prog, Q3 PMF250XNEX, U1 ESP32-PICO-MINI-02, U2 LMR16006+FB

Commit message: Update
Routing:
- net GND: track 73.5 -> 62.6 mm, vias 5 -> 3
- net +3V3: track 33.9 -> 36.2 mm
- net I: track 17.7 -> 19.5 mm
- net O: track 21.6 -> 22.3 mm

Commit message: General tidy of PCB
Parts:
- moved C1 2.39 mm to (97.3, 48.6), turned to 90 degrees
- moved R4 1.45 mm to (95.3, 48.1)
- moved C5 1.42 mm to (95.3, 49.4)
- moved Q3 0.59 mm to (104.0, 48.4), turned to 0 degrees
- moved C2 0.22 mm to (101.8, 41.8)
- moved C3 0.22 mm to (100.5, 45.0)
- moved C4 0.22 mm to (94.2, 45.0)
- moved D1 0.22 mm to (104.7, 42.1)
- moved J2 0.22 mm to (99.8, 56.3)
- moved L1 0.22 mm to (95.8, 41.5)
- moved R1 0.22 mm to (103.1, 44.6)
- moved R2 0.22 mm to (104.3, 44.6)
- moved R5 0.22 mm to (104.8, 39.4)
- moved R6 0.22 mm to (102.3, 39.4)
- moved U1 0.22 mm to (99.8, 44.1)
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Routing:
- net GND: track 62.6 -> 51.0 mm, vias 3 -> 2
- net Net-(J1-Pad4): track 7.43 -> 2.56 mm
- net RX: track 3.87 -> 6.79 mm
- net I: track 19.5 -> 21.9 mm
- net EN: track 6.58 -> 8.55 mm
- net O: track 22.3 -> 20.8 mm
Other:
- outline, holes or cut-outs redrawn
- board text added: "Daikin WiFi"
- board text removed: "Daikin"

Commit message: updated
Parts:
- C2: footprint RevK:Hidden -> RevK:C_0603_
- C3, C4: footprint RevK:Hidden -> RevK:C_0805_
- D2: footprint RevK:Hidden -> RevK:D_1206_
- L1: footprint RevK:Hidden -> RevK:L_4x4_
- U2: footprint RevK:RegulatorBlockFB -> RevK:SOT-23-Thin-6-Reg
- moved J1 0.06 mm to (99.8, 51.4)
- turned D2 to 180 degrees
