File: KiCad/Daikin.kicad_pcb (KiCad board)
At the start: 2 copper layers, 13.2 x 19.5 mm, 19 parts, among them J1 SPOX, J2 Prog, Q3 PMF250XNEX, U1 ESP32-PICO-MINI-02, U2 LMR16006+FB

Commit message: Note on regulator
Parts:
- added ?: , RevK:PasteDaikin, F.Cu at (91.3, 66.4)
Changed lines of the file:
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@@
   (net 37 "O")
   (net 38 "Net-(J1-Pad4)")
+  (footprint "RevK:PasteDaikin" (layer "F.Cu")
+    (at 91.35 66.4)
+    (attr exclude_from_pos_files exclude_from_bom)
+    (fp_text reference "" (at 0 0) (layer "F.SilkS")
+      (effects (font (size 1.27 1.27) (thickness 0.15)))
+    )
+    (fp_text value "" (at 0 0) (layer "F.SilkS")
+      (effects (font (size 1.27 1.27) (thickness 0.15)))
+    )
+    (pad "" smd circle locked (at 0.255 0.255) (size 0.45 0.45) (layers "F.Paste"))
+    (pad "" smd circle locked (at 2.295 0.765) (size 0.45 0.45) (layers "F.Paste"))
+    (pad "" smd circle locked (at 0.255 0.765) (size 0.45 0.45) (layers "F.Paste"))
+    (pad "" smd circle locked (at 7.395 2.295) (size 0.45 0.45) (layers "F.Paste"))
+    (pad "" smd circle locked (at 6.885 1.275) (size 0.45 0.45) (layers "F.Paste"))
+    (pad "" smd circle locked (at 7.395 0.255) (size 0.45 0.45) (layers "F.Paste"))
+    (pad "" smd circle locked (at 13.005 1.275) (size 0.45 0.45) (layers "F.Paste"))
+    (pad "" smd circle locked (at 13.515 1.785) (size 0.45 0.45) (layers "F.Paste"))
+    (pad "" smd circle locked (at 15.555 1.785) (size 0.45 0.45) (layers "F.Paste"))
+    (pad "" smd circle locked (at 0.255 2.295) (size 0.45 0.45) (layers "F.Paste"))
+    (pad "" smd circle locked (at 16.065 1.275) (size 0.45 0.45) (layers "F.Paste"))
+    (pad "" smd circle locked (at 13.515 1.275) (size 0.45 0.45) (layers "F.Paste"))
+    (pad "" smd circle locked (at 2.295 2.295) (size 0.45 0.45) (layers "F.Paste"))
+    (pad "" smd circle locked (at 2.295 1.275) (size 0.45 0.45) (layers "F.Paste"))
+    (pad "" smd circle locked (at 4.845 2.295) (size 0.45 0.45) (layers "F.Paste"))
+    (pad "" smd circle locked (at 16.575 1.275) (size 0.45 0.45) (layers "F.Paste"))
+    (pad "" smd circle locked (at 4.335 1.275) (size 0.45 0.45) (layers "F.Paste"))
+    (pad "" smd circle locked (at 7.905 3.315) (size 0.45 0.45) (layers "F.Paste"))
+    (pad "" smd circle locked (at 1.785 0.255) (size 0.45 0.45) (layers "F.Paste"))
+    (pad "" smd circle locked (at 0.255 3.315) (size 0.45 0.45) (layers "F.Paste"))
+    (pad "" smd circle locked (at 9.945 0.255) (size 0.45 0.45) (layers "F.Paste"))
+    (pad "" smd circle locked (at 9.945 2.295) (size 0.45 0.45) (layers "F.Paste"))
+    (pad "" smd circle locked (at 2.295 1.785) (size 0.45 0.45) (layers "F.Paste"))
+    (pad "" smd circle locked (at 13.515 2.295) (size 0.45 0.45) (layers "F.Paste"))
+    (pad "" smd circle locked (at 17.595 2.295) (size 0.45 0.45) (layers "F.Paste"))
+    (pad "" smd circle locked (at 0.765 3.315) (size 0.45 0.45) (layers "F.Paste"))
+    (pad "" smd circle locked (at 3.315 2.805) (size 0.45 0.45) (layers "F.Paste"))
+    (pad "" smd circle locked (at 4.845 3.315) (size 0.45 0.45) (layers "F.Paste"))
+    (pad "" smd circle locked (at 11.475 1.275) (size 0.45 0.45) (layers "F.Paste"))
+    (pad "" smd circle locked (at 9.945 3.315) (size 0.45 0.45) (layers "F.Paste"))
+    (pad "" smd circle locked (at 1.275 3.315) (size 0.45 0.45) (layers "F.Paste"))
+    (pad "" smd circle locked (at 17.595 2.805) (size 0.45 0.45) (layers "F.Paste"))
+    (pad "" smd circle locked (at 17.595 1.785) (size 0.45 0.45) (layers "F.Paste"))
+    (pad "" smd circle locked (at 2.295 2.805) (size 0.45 0.45) (layers "F.Paste"))
+    (pad "" smd circle locked (at 1.785 3.315) (size 0.45 0.45) (layers "F.Paste"))
+    (pad "" smd circle locked (at 17.085 1.275) (size 0.45 0.45) (layers "F.Paste"))
+    (pad "" smd circle locked (at 13.515 0.255) (size 0.45 0.45) (layers "F.Paste"))
+    (pad "" smd circle locked (at 6.885 3.315) (size 0.45 0.45) (layers "F.Paste"))
+    (pad "" smd circle locked (at 10.455 2.295) (size 0.45 0.45) (layers "F.Paste"))
+    (pad "" smd circle locked (at 9.945 2.805) (size 0.45 0.45) (layers "F.Paste"))
+    (pad "" smd circle locked (at 0.255 1.785) (size 0.45 0.45) (layers "F.Paste"))
+    (pad "" smd circle locked (at 15.555 1.275) (size 0.45 0.45) (layers "F.Paste"))
+    (pad "" smd circle locked (at 11.475 3.315) (size 0.45 0.45) (layers "F.Paste"))
+    (pad "" smd circle locked (at 5.355 2.295) (size 0.45 0.45) (layers "F.Paste"))
+    (pad "" smd circle locked (at 15.555 3.315) (size 0.45 0.45) (layers "F.Paste"))
+    (pad "" smd circle locked (at 4.335 2.295) (size 0.45 0.45) (layers "F.Paste"))
+    (pad "" smd circle locked (at 0.255 1.275) (size 0.45 0.45) (layers "F.Paste"))
+    (pad "" smd circle locked (at 7.395 1.275) (size 0.45 0.45) (layers "F.Paste"))
+    (pad "" smd circle locked (at 9.945 0.765) (size 0.45 0.45) (layers "F.Paste"))
+    (pad "" smd circle locked (at 13.005 3.315) (size 0.45 0.45) (layers "F.Paste"))
+    (pad "" smd circle locked (at 5.355 2.805) (size 0.45 0.45) (layers "F.Paste"))
+    (pad "" smd circle locked (at 5.355 1.785) (size 0.45 0.45) (layers "F.Paste"))
+    (pad "" smd circle locked (at 15.555 2.805) (size 0.45 0.45) (layers "F.Paste"))
+    (pad "" smd circle locked (at 0.255 2.805) (size 0.45 0.45) (layers "F.Paste"))
+    (pad "" smd circle locked (at 5.355 3.315) (size 0.45 0.45) (layers "F.Paste"))
+    (pad "" smd circle locked (at 10.965 2.805) (size 0.45 0.45) (layers "F.Paste"))
+    (pad "" smd circle locked (at 4.845 1.275) (size 0.45 0.45) (layers "F.Paste"))
+    (pad "" smd circle locked (at 17.595 3.315) (size 0.45 0.45) (layers "F.Paste"))
+    (pad "" smd circle locked (at 9.945 1.785) (size 0.45 0.45) (layers "F.Paste"))
+    (pad "" smd circle locked (at 7.395 2.805) (size 0.45 0.45) (layers "F.Paste"))
+    (pad "" smd circle locked (at 1.275 0.255) (size 0.45 0.45) (layers "F.Paste"))
+    (pad "" smd circle locked (at 0.765 0.255) (size 0.45 0.45) (layers "F.Paste"))
+    (pad "" smd circle locked (at 15.555 2.295) (size 0.45 0.45) (layers "F.Paste"))
+    (pad "" smd circle locked (at 3.825 2.295) (size 0.45 0.45) (layers "F.Paste"))
+    (pad "" smd circle locked (at 4.335 3.315) (size 0.45 0.45) (layers "F.Paste"))
+    (pad "" smd circle locked (at 10.965 1.785) (size 0.45 0.45) (layers "F.Paste"))
+    (pad "" smd circle locked (at 13.515 2.805) (size 0.45 0.45) (layers "F.Paste"))
+    (pad "" smd circle locked (at 14.025 3.315) (size 0.45 0.45) (layers "F.Paste"))
+    (pad "" smd circle locked (at 7.395 3.315) (size 0.45 0.45) (layers "F.Paste"))
+    (pad "" smd circle locked (at 3.825 1.275) (size 0.45 0.45) (layers "F.Paste"))
+    (pad "" smd circle locked (at 7.395 1.785) (size 0.45 0.45) (layers "F.Paste"))
+    (pad "" smd circle locked (at 13.515 3.315) (size 0.45 0.45) (layers "F.Paste"))
+    (pad "" smd circle locked (at 3.825 3.315) (size 0.45 0.45) (layers "F.Paste"))
+    (pad "" smd circle locked (at 9.945 1.275) (size 0.45 0.45) (layers "F.Paste"))
+  )
   (footprint "RevK:ESP32-PICO-MINI-02" (layer "F.Cu")
     (at 99.8 44.09325)
@@
     (fp_line (start -6.2 6.6) (end -6.2 -1.3) (layer "F.Fab") (width 0.12))
     (fp_line (start 0 2) (end 1 3) (layer "F.Fab") (width 0.12))
-    (pad "1" thru_hole roundrect (at -3.75 0) (size 1.7 1.85) (drill 0.85) (layers *.Cu *.Mask) (roundrect_rratio 0.147059)
+    (pad "1" thru_hole roundrect (at -3.75 0) (size 1.7 1.85) (drill 0.85) (layers *.Cu *.Mask) (roundrect_rratio 0.1470588235)
       (net 1 "GND") (pinfunction "Pin_1") (pintype "passive"))
     (pad "2" thru_hole oval (at -1.25 0) (size 1.7 1.85) (drill 0.85) (layers *.Cu *.Mask)
@@
       (options (clearance outline) (anchor rect))
       (primitives
-    (gr_arc (start 0.001745 0.000002) (mid 0.707107 0.292894) (end 0.999998 0.998256) (width 0.5))
+    (gr_arc (start 0.001745 0.000002) (mid 0.707106 0.292893) (end 0.999998 0.998254) (width 0.5))
       ))
     (pad "3" smd custom (at -1.1 -4.5 180) (size 0.1 0.1) (layers "B.Cu")
