File: KiCad/Daikin.kicad_sch (KiCad schematic)
At the start: 19 parts, among them J1 SPOX, J2 Prog, Q3 PMF250XNEX, U1 ESP32-PICO-MINI-02, U2 LMR16006+FB

Commit message: General tidy of PCB
Changed lines of the file:
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@@
   (junction (at 147.32 45.72) (diameter 0) (color 0 0 0 0)
+  )
+  (junction (at 50.8 43.18) (diameter 0) (color 0 0 0 0)
   )
   (junction (at 50.8 27.94) (diameter 0) (color 0 0 0 0)
@@
   )
   (wire (pts (xy 144.145 45.72) (xy 147.32 45.72))
+    (stroke (width 0) (type default) (color 0 0 0 0))
+  )
+  (wire (pts (xy 48.26 43.18) (xy 50.8 43.18))
     (stroke (width 0) (type default) (color 0 0 0 0))
   )
@@
     )
   )
-  (global_label "EN" (shape input) (at 50.8 43.18 180) (fields_autoplaced)
+  (global_label "EN" (shape input) (at 48.26 43.18 180) (fields_autoplaced)
     (effects (font (size 1.27 1.27)) (justify right))
-    (property "Intersheet References" "${INTERSHEET_REFS}" (id 0) (at 29.845 1.27 0)
+    (property "Intersheet References" "${INTERSHEET_REFS}" (id 0) (at 27.305 1.27 0)
       (effects (font (size 1.27 1.27)) hide)
     )

Commit message: updated
Parts:
- C1: Part No (none) -> 0603-10nF-50V
- C2: footprint RevK:Hidden -> RevK:C_0603_; Part No (none) -> 0603-100nF-50V
- C3: footprint RevK:Hidden -> RevK:C_0805_; Part No (none) -> 0805-2.2uF-25V
- C4: footprint RevK:Hidden -> RevK:C_0805_; Part No (none) -> 0805-10uF-16V
- C5: Part No (none) -> 0603-100nF-25V
- D2: footprint RevK:Hidden -> RevK:D_1206_
- J1: Part No (none) -> 22057025
- J2: now left out of the parts list
- L1: footprint RevK:Hidden -> RevK:L_4x4_; Part No TYA4020 -> TYA40206R8M-10
- Q3: Part No (none) -> PMF250XNEX
- R1: Part No (none) -> 0603-680R
- R2: Part No (none) -> 0603-2K
- R3: Part No (none) -> 0603-220R
- R4: Part No (none) -> 0603-10K
- R5: Part No (none) -> 0603-100k
- R6: Part No (none) -> 0603-30k
- U1: Part No (none) -> ESP32-PICO-MINI-02-N8R2
- U2: footprint RevK:RegulatorBlockFB -> RevK:SOT-23-Thin-6-Reg
Changed lines of the file:
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@@
       (effects (font (size 1.27 1.27)) (justify right))
     )
-    (property "Footprint" "RevK:Hidden" (id 2) (at 162.56 35.56 0)
+    (property "Footprint" "RevK:C_0603_" (id 2) (at 162.56 35.56 0)
       (effects (font (size 1.27 1.27)) hide)
     )
@@
       (effects (font (size 1.27 1.27)) hide)
     )
-    (property "Part No" "" (id 5) (at 162.56 35.56 0)
+    (property "Part No" "0603-100nF-50V" (id 5) (at 162.56 35.56 0)
       (effects (font (size 1.27 1.27)) hide)
     )
@@
       (effects (font (size 1.27 1.27)) (justify right))
     )
-    (property "Footprint" "RevK:Hidden" (id 2) (at 162.56 37.465 0)
+    (property "Footprint" "RevK:C_0805_" (id 2) (at 162.56 37.465 0)
       (effects (font (size 1.27 1.27)) hide)
     )
@@
       (effects (font (size 1.27 1.27)) hide)
     )
-    (property "Part No" "" (id 5) (at 162.56 37.465 0)
+    (property "Part No" "0805-2.2uF-25V" (id 5) (at 162.56 37.465 0)
       (effects (font (size 1.27 1.27)) hide)
     )
@@
       (effects (font (size 1.27 1.27)) (justify right))
     )
-    (property "Footprint" "RevK:Hidden" (id 2) (at 162.56 39.37 0)
+    (property "Footprint" "RevK:C_0805_" (id 2) (at 162.56 39.37 0)
       (effects (font (size 1.27 1.27)) hide)
     )
@@
       (effects (font (size 1.27 1.27)) hide)
     )
-    (property "Part No" "" (id 5) (at 162.56 39.37 0)
+    (property "Part No" "0805-10uF-16V" (id 5) (at 162.56 39.37 0)
       (effects (font (size 1.27 1.27)) hide)
     )
@@
       (effects (font (size 1.27 1.27)) (justify right))
     )
-    (property "Footprint" "RevK:Hidden" (id 2) (at 162.56 41.275 0)
+    (property "Footprint" "RevK:L_4x4_" (id 2) (at 162.56 41.275 0)
       (effects (font (size 1.27 1.27)) hide)
     )
@@
       (effects (font (size 1.27 1.27)) hide)
     )
-    (property "Part No" "TYA4020" (id 5) (at 162.56 41.275 0)
+    (property "Part No" "TYA40206R8M-10" (id 5) (at 162.56 41.275 0)
       (effects (font (size 1.27 1.27)) hide)
     )
@@
       (effects (font (size 1.27 1.27)) (justify right))
     )
-    (property "Footprint" "RevK:Hidden" (id 2) (at 162.56 43.18 0)
+    (property "Footprint" "RevK:D_1206_" (id 2) (at 162.56 43.18 0)
       (effects (font (size 1.27 1.27)) hide)
     )
@@
       (effects (font (size 1.27 1.27)) hide)
     )
+    (property "Part No" "0603-680R" (id 4) (at 57.15 111.76 90)
+      (effects (font (size 1.27 1.27)) hide)
+    )
     (pin "1")
     (pin "2")
@@
       (effects (font (size 1.27 1.27)) hide)
     )
+    (property "Part No" "0603-10K" (id 4) (at 64.77 27.94 90)
+      (effects (font (size 1.27 1.27)) hide)
+    )
     (pin "1")
     (pin "2")
@@
     )
     (property "Datasheet" "~" (id 3) (at 200.66 41.91 0)
+      (effects (font (size 1.27 1.27)) hide)
+    )
+    (property "Part No" "0603-100nF-25V" (id 4) (at 200.66 41.91 0)
       (effects (font (size 1.27 1.27)) hide)
     )
@@
       (effects (font (size 1.27 1.27)) hide)
     )
+    (property "Part No" "0603-2K" (id 4) (at 57.15 116.84 90)
+      (effects (font (size 1.27 1.27)) hide)
+    )
     (pin "1")
     (pin "2")
@@
       (effects (font (size 1.27 1.27)) (justify left bottom) hide)
     )
+    (property "Part No" "ESP32-PICO-MINI-02-N8R2" (id 8) (at 66.04 66.04 0)
+      (effects (font (size 1.27 1.27)) hide)
+    )
+    (pin "1")
     (pin "1")
     (pin "10")
@@
     (pin "22")
     (pin "23")
+    (pin "23")
     (pin "24")
     (pin "25")
@@
     (pin "28")
     (pin "29")
+    (pin "3")
     (pin "3")
     (pin "30")
@@
       (effects (font (size 1.27 1.27)) hide)
     )
+    (property "Part No" "0603-30k" (id 4) (at 147.32 49.53 90)
+      (effects (font (size 1.27 1.27)) hide)
+    )
     (pin "1")
     (pin "2")
@@
       (effects (font (size 1.27 1.27)) hide)
     )
+    (property "Part No" "0603-10nF-50V" (id 4) (at 39.37 27.94 90)
+      (effects (font (size 1.27 1.27)) hide)
+    )
     (pin "1")
     (pin "2")
@@
     )
     (property "Datasheet" "~" (id 3) (at 147.32 86.36 0)
+      (effects (font (size 1.27 1.27)) hide)
+    )
+    (property "Part No" "22057025" (id 4) (at 147.32 86.36 0)
       (effects (font (size 1.27 1.27)) hide)
     )
@@
       (effects (font (size 1.27 1.27)) (justify left))
     )
-    (property "Footprint" "RevK:RegulatorBlockFB" (id 2) (at 158.75 33.02 0)
+    (property "Footprint" "RevK:SOT-23-Thin-6-Reg" (id 2) (at 158.75 33.02 0)
       (effects (font (size 1.27 1.27)) hide)
     )
@@
       (effects (font (size 1.27 1.27)) hide)
     )
+    (property "Part No" "0603-220R" (id 4) (at 57.15 121.92 90)
+      (effects (font (size 1.27 1.27)) hide)
+    )
     (pin "1")
     (pin "2")
@@
       (effects (font (size 1.27 1.27)) hide)
     )
-    (pin "1")
-    (pin "2")
-    (pin "3")
-  )
-  (symbol (lib_id "RevK:Shelly") (at 198.12 86.36 0) (unit 1)
-    (in_bom yes) (on_board yes)
-    (property "Reference" "J2" (id 0) (at 196.85 77.47 0)
-      (effects (font (size 1.27 1.27)) (justify left))
-    )
-    (property "Value" "Prog" (id 1) (at 198.12 96.52 0)
-      (effects (font (size 1.27 1.27)) (justify left))
-    )
-    (property "Footprint" "RevK:Shelly" (id 2) (at 198.12 95.25 0)
-      (effects (font (size 1.27 1.27)) hide)
-    )
-    (property "Datasheet" "~" (id 3) (at 198.12 95.25 0)
-      (effects (font (size 1.27 1.27)) hide)
-    )
-    (pin "1")
-    (pin "2")
-    (pin "3")
+    (property "Part No" "PMF250XNEX" (id 4) (at 124.46 91.44 0)
+      (effects (font (size 1.27 1.27)) hide)
+    )
+    (pin "1")
+    (pin "2")
+    (pin "3")
+  )
+  (symbol (lib_id "RevK:Shelly") (at 195.58 86.36 0) (unit 1)
+    (in_bom no) (on_board yes)
+    (property "Reference" "J2" (id 0) (at 194.31 77.47 0)
+      (effects (font (size 1.27 1.27)) (justify left))
+    )
+    (property "Value" "Prog" (id 1) (at 195.58 96.52 0)
+      (effects (font (size 1.27 1.27)) (justify left))
+    )
+    (property "Footprint" "RevK:Shelly" (id 2) (at 195.58 95.25 0)
+      (effects (font (size 1.27 1.27)) hide)
+    )
+    (property "Datasheet" "~" (id 3) (at 195.58 95.25 0)
+      (effects (font (size 1.27 1.27)) hide)
+    )
+    (property "Part No" "" (id 4) (at 195.58 86.36 0)
+      (effects (font (size 1.27 1.27)) hide)
+    )
+    (pin "1")
+    (pin "1")
+    (pin "2")
+    (pin "2")
+    (pin "3")
+    (pin "3")
+    (pin "4")
     (pin "4")
     (pin "5")
+    (pin "5")
   )
   (symbol (lib_id "power:+3.3V") (at 193.04 86.36 90) (unit 1)
@@
     )
     (property "Datasheet" "~" (id 3) (at 140.335 45.72 0)
+      (effects (font (size 1.27 1.27)) hide)
+    )
+    (property "Part No" "0603-100k" (id 4) (at 140.335 45.72 90)
       (effects (font (size 1.27 1.27)) hide)
     )
@@
     )
     (path "/00000000-0000-0000-0000-0000610f9b88"
-      (reference "C2") (unit 1) (value "0.1uF") (footprint "RevK:Hidden")
+      (reference "C2") (unit 1) (value "0.1uF") (footprint "RevK:C_0603_")
     )
     (path "/00000000-0000-0000-0000-0000610fd0ef"
-      (reference "C3") (unit 1) (value "2.2uF") (footprint "RevK:Hidden")
+      (reference "C3") (unit 1) (value "2.2uF") (footprint "RevK:C_0805_")
     )
     (path "/00000000-0000-0000-0000-0000610fd80e"
-      (reference "C4") (unit 1) (value "10uF") (footprint "RevK:Hidden")
+      (reference "C4") (unit 1) (value "10uF") (footprint "RevK:C_0805_")
     )
     (path "/296b967f-b7a9-453f-856a-7b874fdca3db"
@@
     )
     (path "/00000000-0000-0000-0000-0000610fe5d2"
-      (reference "D2") (unit 1) (value "Schottky") (footprint "RevK:Hidden")
+      (reference "D2") (unit 1) (value "Schottky") (footprint "RevK:D_1206_")
     )
     (path "/af073fa6-a783-40f2-9751-692984a62ffc"
@@
     )
     (path "/00000000-0000-0000-0000-0000610fe01a"
-      (reference "L1") (unit 1) (value "6.8uH") (footprint "RevK:Hidden")
+      (reference "L1") (unit 1) (value "6.8uH") (footprint "RevK:L_4x4_")
     )
     (path "/ebcfdf36-110d-4f79-9de0-e4fcd76c1d6e"
@@
     )
     (path "/c88f1737-32b5-4cea-a76f-93ad322556d3"
-      (reference "U2") (unit 1) (value "LMR16006+FB") (footprint "RevK:RegulatorBlockFB")
-    )
-  )
+      (reference "U2") (unit 1) (value "LMR16006+FB") (footprint "RevK:SOT-23-Thin-6-Reg")
+    )
+  )

Commit message: Cleaner defaults
Other:
- note added: "User either variable LMR16006 with 100k/30k Or fixed 3.3V LMR16006 Q3 part with 0R/NF"
Changed lines of the file:
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@@
+    (effects (font (size 1.27 1.27)) (justify left bottom))
+  )
+  (text "User either variable LMR16006 with 100k/30k\nOr fixed 3.3V LMR16006 Q3 part with 0R/NF"
+    (at 152.4 55.88 0)
     (effects (font (size 1.27 1.27)) (justify left bottom))
   )

Commit message: Note on regulator
Other:
- note added: "Note, a better regulator for this may be the TLV62569PDDC or TLV62569PDRL as it is suitable up to 5.5V input and small footprint and power good out."
- note removed: "User either variable LMR16006 with 100k/30k Or fixed 3.3V LMR16006 Q3 part with 0R/NF"
Changed lines of the file:
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@@
     (effects (font (size 1.27 1.27)) (justify left bottom))
   )
-  (text "User either variable LMR16006 with 100k/30k\nOr fixed 3.3V LMR16006 Q3 part with 0R/NF"
-    (at 152.4 55.88 0)
+  (text "Note, a better regulator for this may be the TLV62569PDDC or TLV62569PDRL as it is suitable up to 5.5V input and small footprint and power good out."
+    (at 106.045 120.65 0)
     (effects (font (size 1.27 1.27)) (justify left bottom))
   )
