File: PCB/Daikin/Daikin.kicad_pcb (KiCad board)
At the start: 2 copper layers, 13.2 x 19.5 mm, 19 parts, among them J1 1x4, J2 Prog, Q3 PMF250XNEX, U1 ESP32-PICO-MINI-02, U2 LMR16006XDDCR

Commit message: Tidy
Changed lines of the file:
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@@
       (options (clearance outline) (anchor rect))
       (primitives
-    (gr_arc (start 0.001745 0.000002) (mid 0.707106 0.292893) (end 0.999998 0.998254) (width 0.5))
+    (gr_arc (start 0.001745 0.000002) (mid 0.706489 0.292277) (end 0.999993 0.996509) (width 0.5))
       ))
     (pad "6" smd rect (at 0.95 -1.35 90) (size 1.1 0.6) (layers "B.Cu" "B.Paste" "B.Mask")

Commit message: Tidy
Parts:
- U2: value LMR16006XDDCR -> LMR16006YDDCR

Commit message: Faikin
Other:
- board text added: "Faikin WiFi"
- board text removed: "Daikin WiFi"
Changed lines of the file:
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@@
       (options (clearance outline) (anchor rect))
       (primitives
-    (gr_arc (start 0.001745 0.000002) (mid 0.707723 0.293511) (end 1 1) (width 0.5))
+    (gr_arc (start 0.001745 0.000002) (mid 0.707107 0.292894) (end 0.999998 0.998256) (width 0.5))
       ))
     (pad "5" smd rect (at 0 -1.35 90) (size 1.1 0.6) (layers "B.Cu" "B.Paste" "B.Mask")
@@
     (effects (font (size 0.5 0.5) (thickness 0.08)) (justify mirror))
   )
-  (gr_text "Daikin\nWiFi" (at 100.2 48.9) (layer "B.SilkS")
+  (gr_text "Faikin\nWiFi" (at 100.2 48.9) (layer "B.SilkS")
     (effects (font (size 0.75 0.75) (thickness 0.1)) (justify mirror))
   )
