File: PCB/Daikin/Daikin.kicad_pcb (KiCad board)
At the start: 2 copper layers, 15.2 x 20 mm, 22 parts, among them J1 1x5, J2 Prog, Q3 PMF250XNEX, U1 ESP32-PICO-MINI-02, U2 LMR16006YDDCR

Commit message: Date
Other:
- board text added: "${DATE}"
Changed lines of the file:
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@@
   (gr_arc (start 92.4 39.5) (mid 92.692893 38.792893) (end 93.4 38.5) (layer "Edge.Cuts") (width 0.1))
   (gr_line (start 93.4 38.5) (end 106.6 38.5) (layer "Edge.Cuts") (width 0.1))
-  (gr_text "26" (at 99.86 53.4) (layer "B.SilkS")
-    (effects (font (size 0.6 0.6) (thickness 0.1)) (justify mirror))
+  (gr_text "26" (at 100 53.4) (layer "B.SilkS")
+    (effects (font (size 0.75 0.75) (thickness 0.1)) (justify mirror))
   )
-  (gr_text "NC" (at 104.94 53.4) (layer "B.SilkS")
-    (effects (font (size 0.6 0.6) (thickness 0.1)) (justify mirror))
+  (gr_text "NC" (at 105 53.4) (layer "B.SilkS")
+    (effects (font (size 0.75 0.75) (thickness 0.1)) (justify mirror))
   )
-  (gr_text "⏚" (at 94.78 53.4) (layer "B.SilkS")
-    (effects (font (size 0.6 0.6) (thickness 0.1)) (justify mirror))
+  (gr_text "⏚" (at 95 53.4) (layer "B.SilkS")
+    (effects (font (size 0.75 0.75) (thickness 0.1)) (justify mirror))
   )
   (gr_text "8/19/7" (at 104.1 41.7 90) (layer "B.SilkS")
     (effects (font (size 0.5 0.5) (thickness 0.08)) (justify mirror))
   )
-  (gr_text "↑" (at 103.26 53.35) (layer "B.SilkS")
+  (gr_text "↑" (at 103.2 50.7) (layer "B.SilkS")
     (effects (font (size 0.5 0.5) (thickness 0.08)) (justify mirror))
   )
-  (gr_text "DC" (at 97.32 53.4) (layer "B.SilkS")
-    (effects (font (size 0.6 0.6) (thickness 0.1)) (justify mirror))
+  (gr_text "DC" (at 97.5 53.4) (layer "B.SilkS")
+    (effects (font (size 0.75 0.75) (thickness 0.1)) (justify mirror))
   )
-  (gr_text "27" (at 102.4 53.4) (layer "B.SilkS")
-    (effects (font (size 0.6 0.6) (thickness 0.1)) (justify mirror))
+  (gr_text "27" (at 102.5 53.4) (layer "B.SilkS")
+    (effects (font (size 0.75 0.75) (thickness 0.1)) (justify mirror))
   )
   (gr_text "Faikin - www.me.uk" (at 100 55) (layer "B.SilkS")
     (effects (font (size 0.9 0.9) (thickness 0.15)) (justify mirror))
   )
-  (gr_text "↓" (at 100.76 53.35) (layer "B.SilkS")
+  (gr_text "↓" (at 99.2 50.7) (layer "B.SilkS")
     (effects (font (size 0.5 0.5) (thickness 0.08)) (justify mirror))
   )
+  (gr_text "${DATE}" (at 93.2 43.7 90) (layer "B.SilkS")
+    (effects (font (size 0.8 0.8) (thickness 0.15)) (justify mirror))
+  )
   (dimension (type aligned) (layer "Dwgs.User")

Commit message: Tweak
Other:
- outline, holes or cut-outs redrawn
- board text added: "faikin.revk.uk"
- board text removed: "Faikin - www.me.uk"
Changed lines of the file:
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@@
     )
   )
-  (property "DATE" "2023-03-29")
+  (property "DATE" "2023-03-31")
   (net 0 "")
   (net 1 "GND")
@@
       (net 37 "Net-(J2-Pad5)") (pinfunction "Tx") (pintype "passive"))
   )
-  (gr_line (start 107.6 39.5) (end 107.6 58.5) (layer "Edge.Cuts") (width 0.1))
-  (gr_arc (start 106.6 38.5) (mid 107.307107 38.792893) (end 107.6 39.5) (layer "Edge.Cuts") (width 0.1))
+  (gr_line (start 93.4 38.5) (end 92.4 50.2) (layer "Edge.Cuts") (width 0.1))
+  (gr_line (start 107.6 50.2) (end 107.6 58.5) (layer "Edge.Cuts") (width 0.1))
+  (gr_line (start 106.6 38.5) (end 107.6 50.2) (layer "Edge.Cuts") (width 0.1))
   (gr_line (start 107.6 58.5) (end 92.4 58.5) (layer "Edge.Cuts") (width 0.1))
-  (gr_line (start 92.4 58.5) (end 92.4 39.5) (layer "Edge.Cuts") (width 0.1))
-  (gr_arc (start 92.4 39.5) (mid 92.692893 38.792893) (end 93.4 38.5) (layer "Edge.Cuts") (width 0.1))
+  (gr_line (start 92.4 58.5) (end 92.4 50.2) (layer "Edge.Cuts") (width 0.1))
   (gr_line (start 93.4 38.5) (end 106.6 38.5) (layer "Edge.Cuts") (width 0.1))
   (gr_text "26" (at 100 53.4) (layer "B.SilkS")
@@
     (effects (font (size 0.75 0.75) (thickness 0.1)) (justify mirror))
   )
-  (gr_text "Faikin - www.me.uk" (at 100 55) (layer "B.SilkS")
-    (effects (font (size 0.9 0.9) (thickness 0.15)) (justify mirror))
+  (gr_text "faikin.revk.uk" (at 100 55) (layer "B.SilkS")
+    (effects (font (size 1 1) (thickness 0.15)) (justify mirror))
   )
   (gr_text "↓" (at 99.2 50.7) (layer "B.SilkS")
     (effects (font (size 0.5 0.5) (thickness 0.08)) (justify mirror))
   )
-  (gr_text "${DATE}" (at 93.2 43.7 90) (layer "B.SilkS")
-    (effects (font (size 0.8 0.8) (thickness 0.15)) (justify mirror))
+  (gr_text "${DATE}" (at 100.3 50.3) (layer "F.SilkS")
+    (effects (font (size 0.8 0.8) (thickness 0.15)))
   )
   (dimension (type aligned) (layer "Dwgs.User")

Commit message: Revised for production
Routing:
- net Net-(J2-Pad4): track 20.0 -> 19.5 mm
Changed lines of the file:
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@@
     )
   )
-  (property "DATE" "2023-03-31")
+  (property "DATE" "2023-04-08")
   (net 0 "")
   (net 1 "GND")
@@
     (descr "Capacitor SMD 0603 (1608 Metric), square (rectangular) end terminal, IPC_7351 nominal, (Body size source: IPC-SM-782 page 76, https://www.pcb-3d.com/wordpress/wp-content/uploads/ipc-sm-782a_amendment_1_and_2.pdf), generated with kicad-footprint-generator")
     (tags "capacitor")
+    (property "JLCPCB Rotation Offset" "90")
     (property "Manufacturer" "")
     (property "Note" "")
@@
   (arc (start 105.80675 44) (mid 105.872688 44.027312) (end 105.9 44.09325) (width 0.25) (layer "F.Cu") (net 36))
   (arc (start 104.05 44.585704) (mid 104.221549 44.171549) (end 104.635704 44) (width 0.25) (layer "F.Cu") (net 36))
+  (segment (start 104.7 47.2) (end 104.875736 47.2) (width 0.25) (layer "B.Cu") (net 36))
+  (segment (start 106.7 51.3) (end 106.7 50.155634) (width 0.25) (layer "B.Cu") (net 36))
   (segment (start 105.9 54.2) (end 103.9 54.2) (width 0.25) (layer "B.Cu") (net 36))
-  (segment (start 106.7 53.1) (end 106.7 48.5) (width 0.25) (layer "B.Cu") (net 36))
-  (segment (start 104.5 47.2) (end 105.4 47.2) (width 0.25) (layer "B.Cu") (net 36))
-  (segment (start 106.7 53.1) (end 106.7 53.4) (width 0.25) (layer "B.Cu") (net 36))
-  (arc (start 104 46.7) (mid 104.146447 47.053553) (end 104.5 47.2) (width 0.25) (layer "B.Cu") (net 36))
-  (arc (start 106.7 48.5) (mid 106.319239 47.580761) (end 105.4 47.2) (width 0.25) (layer "B.Cu") (net 36))
+  (segment (start 104 46.7) (end 104.358578 47.058578) (width 0.25) (layer "B.Cu") (net 36))
+  (segment (start 106.7 53.4) (end 106.7 51.3) (width 0.25) (layer "B.Cu") (net 36))
+  (arc (start 106.7 50.155634) (mid 106.414119 48.718415) (end 105.6 47.5) (width 0.25) (layer "B.Cu") (net 36))
+  (arc (start 104.875736 47.2) (mid 105.267704 47.277968) (end 105.6 47.5) (width 0.25) (layer "B.Cu") (net 36))
   (arc (start 106.7 53.4) (mid 106.465685 53.965685) (end 105.9 54.2) (width 0.25) (layer "B.Cu") (net 36))
+  (arc (start 104.358578 47.058578) (mid 104.515224 47.163245) (end 104.7 47.2) (width 0.25) (layer "B.Cu") (net 36))
   (arc (start 103.9 54.2) (mid 103.687868 54.112132) (end 103.6 53.9) (width 0.25) (layer "B.Cu") (net 36))
   (segment (start 103.2 46.94325) (end 103.2 44.7) (width 0.25) (layer "F.Cu") (net 37))
