File: PCB/Daikin/Daikin.kicad_sch (KiCad schematic)
At the start: 19 parts, among them J1 SPOX, J2 Prog, Q3 PMF250XNEX, U1 ESP32-PICO-MINI-02, U2 LMR16006+FB

Commit message: Not finished, working on production files
Parts:
- C2: value 0.1uF -> 100nF; LCSC Part # (none) -> C30926; Part No 0603-100nF-50V -> (none)
- C3: LCSC Part # (none) -> C19110; Part No 0805-2.2uF-25V -> (none)
- C4: LCSC Part # (none) -> C17024; Part No 0805-10uF-16V -> (none)
- D1: LCSC Part # (none) -> C264507
- D2: LCSC Part # (none) -> C143805; Part No CD1206-B2100 -> (none)
- J1: value SPOX -> 1x4; footprint RevK:Molex_MiniSPOX_H4RA -> RevK:JLC-PinHeader_1x04_P2.54mm_Right; LCSC Part # (none) -> C91552; Part No 22057025 -> (none)
- L1: LCSC Part # (none) -> C354575; Manufacturer Laird -> (none); Part No TYA40206R8M-10 -> (none)
- R5: value 100k 1% or 0R -> 100k 1%; LCSC Part # (none) -> C14675; Part No 0603-100k -> (none)
- R6: value 30k 1% or NF -> 30k 1%; LCSC Part # (none) -> C100001; Part No 0603-30k -> (none)
- U1: LCSC Part # (none) -> C2980306
- U2: value LMR16006+FB -> LMR16006XDDCR; LCSC Part # (none) -> C87080
Connections:
- net +3V3 is gone; now on net +3.3V: C5.1, D1.1 (A), J2.3 (3V3), R4.1, R5.1, U1.3 (3V3), U2.4 (VOUT)
- net GPIO0: no longer J2.2 (0), U1.23 (IO0)
- net at U1.23 (IO0): now also J2.2 (0)
- net +3.3V: now reaches U1.3 (3V3)
- net at J2.4 (Rx): now also U1.30 (RXD0)
- net at J2.5 (Tx): now also U1.31 (TXD0)
- removed net I: J2.4 (Rx), U1.30 (RXD0)
- removed net O: J2.5 (Tx), U1.31 (TXD0)
Other:
- note added: "LED part needs sorting in LCSC/JLC Diode wrong way somehow on JLC Change FET as short supply"
- note removed: "Note, a better regulator for this may be the TLV62569PDDC or TLV62569PDRL as it is suitable up to 5.5V input and small footprint and power good out."

Commit message: Parts for JLC
Parts:
- removed D1: RGB, RevK:LED-RGB-1.6x1.6, symbol Device:LED_ARGB
- added D1: LED_BARG, RevK:MHS190RGBCT, symbol Device:LED_BARG
- D2: JLCPCB Rotation Offset (none) -> 180
- Q3: LCSC Part # (none) -> C504047
- R1: value 680R -> 300R
- R2: value 2K -> 1K
- R3: value 220R -> 100R
Connections:
- net +3.3V: now also D1.2 (A)
- net G: now also U1.33 (IO19); no longer U1.28 (IO8)
- net R: now also U1.28 (IO8); no longer U1.33 (IO19)
- net at R1.1: now also D1.3 (RK)
- net at R2.1: now also D1.4 (GK)
- net at R3.1: now also D1.1 (BK)
Other:
- note added: "Needs new LED from LCSC"
- note removed: "LED part needs sorting in LCSC/JLC Diode wrong way somehow on JLC Change FET as short supply"
Changed lines of the file:
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@@
     (effects (font (size 1.27 1.27)) (justify left bottom))
   )
-  (text "LED part needs sorting in LCSC/JLC\nDiode wrong way somehow on JLC\nChange FET as short supply"
-    (at 99.695 143.51 0)
+  (text "Needs new LED from LCSC" (at 99.695 143.51 0)
     (effects (font (size 5 5)) (justify left bottom))
   )
-  (global_label "G" (shape input) (at 50.8 76.2 180) (fields_autoplaced)
-    (effects (font (size 1.27 1.27)) (justify right))
-    (property "Intersheet References" "${INTERSHEET_REFS}" (id 0) (at -52.07 -24.13 0)
-      (effects (font (size 1.27 1.27)) hide)
-    )
-  )
-  (global_label "R" (shape input) (at 81.28 63.5 0) (fields_autoplaced)
+  (global_label "G" (shape input) (at 81.28 63.5 0) (fields_autoplaced)
     (effects (font (size 1.27 1.27)) (justify left))
-    (property "Intersheet References" "${INTERSHEET_REFS}" (id 0) (at 184.15 158.75 0)
+    (property "Intersheet References" "${INTERSHEET_REFS}" (id 0) (at 184.15 163.83 0)
+      (effects (font (size 1.27 1.27)) hide)
+    )
+  )
+  (global_label "R" (shape input) (at 50.8 76.2 180) (fields_autoplaced)
+    (effects (font (size 1.27 1.27)) (justify right))
+    (property "Intersheet References" "${INTERSHEET_REFS}" (id 0) (at -52.07 -19.05 0)
       (effects (font (size 1.27 1.27)) hide)
     )
@@
     (effects (font (size 1.27 1.27)) (justify right))
     (property "Intersheet References" "${INTERSHEET_REFS}" (id 0) (at 117.6908 33.5756 0)
-      (effects (font (size 1.27 1.27)) (justify right) hide)
-    )
-  )
-  (global_label "GPIO0" (shape bidirectional) (at 50.8 63.5 180) (fields_autoplaced)
-    (effects (font (size 1.27 1.27)) (justify right))
-    (property "Intersheet References" "${INTERSHEET_REFS}" (id 0) (at 42.791 63.4206 0)
       (effects (font (size 1.27 1.27)) (justify right) hide)
     )
@@
     (in_bom yes) (on_board yes)
     (property "Reference" "R1" (id 0) (at 57.15 113.665 90))
-    (property "Value" "680R" (id 1) (at 57.15 111.76 90))
+    (property "Value" "300R" (id 1) (at 57.15 111.76 90))
     (property "Footprint" "RevK:R_0603" (id 2) (at 57.15 109.982 90)
       (effects (font (size 1.27 1.27)) hide)
@@
       (effects (font (size 1.27 1.27)) hide)
     )
+    (property "JLCPCB Rotation Offset" "180" (id 7) (at 151.765 40.005 0)
+      (effects (font (size 1.27 1.27)) hide)
+    )
     (pin "~")
   )
@@
     (in_bom yes) (on_board yes)
     (property "Reference" "R2" (id 0) (at 57.15 118.745 90))
-    (property "Value" "2K" (id 1) (at 57.15 116.84 90))
+    (property "Value" "1K" (id 1) (at 57.15 116.84 90))
     (property "Footprint" "RevK:R_0603" (id 2) (at 57.15 115.062 90)
       (effects (font (size 1.27 1.27)) hide)
@@
     (pin "~")
   )
+  (symbol (lib_id "Device:LED_BARG") (at 66.04 116.84 0) (unit 1)
+    (in_bom yes) (on_board yes) (fields_autoplaced)
+    (property "Reference" "D1" (id 0) (at 66.04 104.7582 0))
+    (property "Value" "LED_BARG" (id 1) (at 66.04 107.2951 0))
+    (property "Footprint" "RevK:MHS190RGBCT" (id 2) (at 66.04 118.11 0)
+      (effects (font (size 1.27 1.27)) hide)
+    )
+    (property "Datasheet" "~" (id 3) (at 66.04 118.11 0)
+      (effects (font (size 1.27 1.27)) hide)
+    )
+    (property "LCSC Part #" "C409798" (id 4) (at 66.04 116.84 0)
+      (effects (font (size 1.27 1.27)) hide)
+    )
+    (pin "1")
+    (pin "2")
+    (pin "3")
+    (pin "4")
+  )
   (symbol (lib_name "GND_2") (lib_id "power:GND") (at 121.92 96.52 0) (unit 1)
     (in_bom yes) (on_board yes) (fields_autoplaced)
@@
     (pin "1")
   )
-  (symbol (lib_id "Device:LED_ARGB") (at 66.04 116.84 0) (unit 1)
-    (in_bom yes) (on_board yes)
-    (property "Reference" "D1" (id 0) (at 66.04 104.2162 0))
-    (property "Value" "RGB" (id 1) (at 66.04 106.5276 0))
-    (property "Footprint" "RevK:LED-RGB-1.6x1.6" (id 2) (at 66.04 118.11 0)
-      (effects (font (size 1.27 1.27)) hide)
-    )
-    (property "Datasheet" "~" (id 3) (at 66.04 118.11 0)
-      (effects (font (size 1.27 1.27)) hide)
-    )
-    (property "Manufacturer" "Kingbright" (id 4) (at 66.04 116.84 0)
-      (effects (font (size 1.27 1.27)) hide)
-    )
-    (property "Part No" "APTF1616LSEEZGKQBKC" (id 5) (at 66.04 116.84 0)
-      (effects (font (size 1.27 1.27)) hide)
-    )
-    (property "LCSC Part #" "C264507" (id 6) (at 66.04 116.84 0)
-      (effects (font (size 1.27 1.27)) hide)
-    )
-    (pin "1")
-    (pin "2")
-    (pin "3")
-    (pin "4")
-  )
   (symbol (lib_id "Device:R") (at 132.08 45.72 90) (unit 1)
     (in_bom yes) (on_board yes)
@@
     (in_bom yes) (on_board yes)
     (property "Reference" "R3" (id 0) (at 57.15 123.825 90))
-    (property "Value" "220R" (id 1) (at 57.15 121.92 90))
+    (property "Value" "100R" (id 1) (at 57.15 121.92 90))
     (property "Footprint" "RevK:R_0603" (id 2) (at 57.15 120.142 90)
       (effects (font (size 1.27 1.27)) hide)
@@
     )
     (property "Part No" "PMF250XNEX" (id 4) (at 124.46 91.44 0)
+      (effects (font (size 1.27 1.27)) hide)
+    )
+    (property "LCSC Part #" "C504047" (id 5) (at 124.46 91.44 0)
       (effects (font (size 1.27 1.27)) hide)
     )
@@
       (effects (font (size 1.27 1.27)) (justify left))
     )
-    (property "Value" "Prog" (id 1) (at 81.28 62.23 0)
+    (property "Value" "Prog" (id 1) (at 83.82 47.625 0)
       (effects (font (size 1.27 1.27)) (justify left))
     )
@@
       (reference "C5") (unit 1) (value "100nF") (footprint "RevK:C_0603")
     )
-    (path "/c402b2b8-0bbd-4038-b1b9-845d84949881"
-      (reference "D1") (unit 1) (value "RGB") (footprint "RevK:LED-RGB-1.6x1.6")
+    (path "/a7518107-ce5c-4f9d-bc2d-0e43ac670ca1"
+      (reference "D1") (unit 1) (value "LED_BARG") (footprint "RevK:MHS190RGBCT")
     )
     (path "/2a24d3f6-974c-420b-8ec3-07a5d48dea6b"
@@
     )
     (path "/06b0f59d-5955-4cff-a86d-1a17e2ebba6e"
-      (reference "R1") (unit 1) (value "680R") (footprint "RevK:R_0603")
+      (reference "R1") (unit 1) (value "300R") (footprint "RevK:R_0603")
     )
     (path "/79395739-5b58-4aae-aef4-d23a7b2201c1"
-      (reference "R2") (unit 1) (value "2K") (footprint "RevK:R_0603")
+      (reference "R2") (unit 1) (value "1K") (footprint "RevK:R_0603")
     )
     (path "/d6338c10-d82f-4d48-a66e-2ce47a2f9a18"
-      (reference "R3") (unit 1) (value "220R") (footprint "RevK:R_0603")
+      (reference "R3") (unit 1) (value "100R") (footprint "RevK:R_0603")
     )
     (path "/1f797175-97b5-4fed-b82b-5985f9063700"

Commit message: No change
Parts:
- C2: footprint RevK:C_0603_ -> RevK:Hidden
- C3, C4: footprint RevK:C_0805_ -> RevK:Hidden
- D2: footprint RevK:D_1206_ -> RevK:Hidden
- L1: footprint RevK:L_4x4_ -> RevK:Hidden
- Q3: footprint Package_TO_SOT_SMD:SOT-323_SC-70 -> Package_TO_SOT_SMD:SOT-23
Changed lines of the file:
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@@
       (effects (font (size 1.27 1.27)) (justify right))
     )
-    (property "Footprint" "RevK:C_0805_" (id 2) (at 151.765 34.29 0)
+    (property "Footprint" "RevK:Hidden" (id 2) (at 151.765 34.29 0)
       (effects (font (size 1.27 1.27)) hide)
     )
@@
       (effects (font (size 1.27 1.27)) hide)
     )
+    (property "Part No" "" (id 6) (at 151.765 34.29 0)
+      (effects (font (size 1.27 1.27)) hide)
+    )
     (pin "~")
   )
@@
       (effects (font (size 1.27 1.27)) (justify right))
     )
-    (property "Footprint" "RevK:D_1206_" (id 2) (at 151.765 40.005 0)
+    (property "Footprint" "RevK:Hidden" (id 2) (at 151.765 40.005 0)
       (effects (font (size 1.27 1.27)) hide)
     )
@@
     )
     (property "JLCPCB Rotation Offset" "180" (id 7) (at 151.765 40.005 0)
+      (effects (font (size 1.27 1.27)) hide)
+    )
+    (property "Part No" "" (id 7) (at 151.765 40.005 0)
+      (effects (font (size 1.27 1.27)) hide)
+    )
+    (property "Note" "" (id 8) (at 151.765 40.005 0)
       (effects (font (size 1.27 1.27)) hide)
     )
@@
     (pin "5")
   )
-  (symbol (lib_name "GND_3") (lib_id "power:GND") (at 200.66 45.72 0) (unit 1)
+  (symbol (lib_id "power:GND") (at 200.66 45.72 0) (unit 1)
     (in_bom yes) (on_board yes) (fields_autoplaced)
     (property "Reference" "#PWR0110" (id 0) (at 200.66 52.07 0)
@@
     (pin "9")
   )
-  (symbol (lib_id "power:GND") (at 125.73 45.72 0) (unit 1)
+  (symbol (lib_name "GND_5") (lib_id "power:GND") (at 125.73 45.72 0) (unit 1)
     (in_bom yes) (on_board yes) (fields_autoplaced)
     (property "Reference" "#PWR0101" (id 0) (at 125.73 52.07 0)
@@
       (effects (font (size 1.27 1.27)) (justify right))
     )
-    (property "Footprint" "RevK:C_0805_" (id 2) (at 151.765 36.195 0)
+    (property "Footprint" "RevK:Hidden" (id 2) (at 151.765 36.195 0)
       (effects (font (size 1.27 1.27)) hide)
     )
@@
     )
     (property "LCSC Part #" "C17024" (id 5) (at 151.765 36.195 0)
+      (effects (font (size 1.27 1.27)) hide)
+    )
+    (property "Part No" "" (id 6) (at 151.765 36.195 0)
       (effects (font (size 1.27 1.27)) hide)
     )
@@
     (pin "4")
   )
-  (symbol (lib_name "GND_2") (lib_id "power:GND") (at 121.92 96.52 0) (unit 1)
+  (symbol (lib_id "power:GND") (at 121.92 96.52 0) (unit 1)
     (in_bom yes) (on_board yes) (fields_autoplaced)
     (property "Reference" "#PWR0102" (id 0) (at 121.92 102.87 0)
@@
       (effects (font (size 1.27 1.27)) (justify right))
     )
-    (property "Footprint" "RevK:C_0603_" (id 2) (at 151.765 32.385 0)
+    (property "Footprint" "RevK:Hidden" (id 2) (at 151.765 32.385 0)
       (effects (font (size 1.27 1.27)) hide)
     )
@@
     )
     (property "LCSC Part #" "C30926" (id 5) (at 151.765 32.385 0)
+      (effects (font (size 1.27 1.27)) hide)
+    )
+    (property "Part No" "" (id 6) (at 151.765 32.385 0)
       (effects (font (size 1.27 1.27)) hide)
     )
@@
       (effects (font (size 1.27 1.27)) (justify right))
     )
-    (property "Footprint" "RevK:L_4x4_" (id 2) (at 151.765 38.1 0)
+    (property "Footprint" "RevK:Hidden" (id 2) (at 151.765 38.1 0)
       (effects (font (size 1.27 1.27)) hide)
     )
@@
     )
     (property "LCSC Part #" "C354575" (id 6) (at 151.765 38.1 0)
+      (effects (font (size 1.27 1.27)) hide)
+    )
+    (property "Part No" "" (id 5) (at 151.765 38.1 0)
+      (effects (font (size 1.27 1.27)) hide)
+    )
+    (property "Note" "" (id 6) (at 151.765 38.1 0)
       (effects (font (size 1.27 1.27)) hide)
     )
@@
     (pin "2")
   )
-  (symbol (lib_name "GND_4") (lib_id "power:GND") (at 35.56 27.94 270) (unit 1)
+  (symbol (lib_id "power:GND") (at 35.56 27.94 270) (unit 1)
     (in_bom yes) (on_board yes) (fields_autoplaced)
     (property "Reference" "#PWR0108" (id 0) (at 29.21 27.94 0)
@@
       (effects (font (size 1.27 1.27)) (justify left))
     )
-    (property "Footprint" "Package_TO_SOT_SMD:SOT-323_SC-70" (id 2) (at 119.38 88.9 0)
+    (property "Footprint" "Package_TO_SOT_SMD:SOT-23" (id 2) (at 119.38 88.9 0)
       (effects (font (size 1.27 1.27)) hide)
     )
@@
     )
     (path "/b8671e87-1469-44e2-ab1b-2dbb18ba7eba"
-      (reference "C2") (unit 1) (value "100nF") (footprint "RevK:C_0603_")
+      (reference "C2") (unit 1) (value "100nF") (footprint "RevK:Hidden")
     )
     (path "/235f276c-84a0-4d76-963d-c6858a80fc70"
-      (reference "C3") (unit 1) (value "2.2uF") (footprint "RevK:C_0805_")
+      (reference "C3") (unit 1) (value "2.2uF") (footprint "RevK:Hidden")
     )
     (path "/9cc8d907-ad75-4ab2-9d9f-0dfdb290d4b7"
-      (reference "C4") (unit 1) (value "10uF") (footprint "RevK:C_0805_")
+      (reference "C4") (unit 1) (value "10uF") (footprint "RevK:Hidden")
     )
     (path "/296b967f-b7a9-453f-856a-7b874fdca3db"
@@
     )
     (path "/2a24d3f6-974c-420b-8ec3-07a5d48dea6b"
-      (reference "D2") (unit 1) (value "Schottky") (footprint "RevK:D_1206_")
+      (reference "D2") (unit 1) (value "Schottky") (footprint "RevK:Hidden")
     )
     (path "/af073fa6-a783-40f2-9751-692984a62ffc"
@@
     )
     (path "/bbd07ae0-123b-41d3-a93c-85b702312370"
-      (reference "L1") (unit 1) (value "6.8uH") (footprint "RevK:L_4x4_")
+      (reference "L1") (unit 1) (value "6.8uH") (footprint "RevK:Hidden")
     )
     (path "/ebcfdf36-110d-4f79-9de0-e4fcd76c1d6e"
-      (reference "Q3") (unit 1) (value "PMF250XNEX") (footprint "Package_TO_SOT_SMD:SOT-323_SC-70")
+      (reference "Q3") (unit 1) (value "PMF250XNEX") (footprint "Package_TO_SOT_SMD:SOT-23")
     )
     (path "/06b0f59d-5955-4cff-a86d-1a17e2ebba6e"
