File: PCB/Daikin/Daikin.kicad_sch (KiCad schematic)
At the start: 19 parts, among them J1 1x4, J2 Prog, Q3 PMF250XNEX, U1 ESP32-PICO-MINI-02, U2 LMR16006XDDCR

Commit message: Corrected production files
Parts:
- removed U2: LMR16006XDDCR, RevK:SOT-23-Thin-6-Reg, symbol RevK:LMR16006+FB
- added U2: LMR16006XDDCR, RevK:SOT-23-Thin-6-Reg, symbol RevK:LMR16006XDDCR
- C2: footprint RevK:Hidden -> RevK:C_0603_
- C3, C4: footprint RevK:Hidden -> RevK:C_0805_; Note 0603 or 0805 -> (none)
- D2: footprint RevK:Hidden -> RevK:D_1206_
- L1: footprint RevK:Hidden -> RevK:L_4x4_
- Q3: footprint Package_TO_SOT_SMD:SOT-23 -> RevK:SOT-323_SC-70; JLCPCB Rotation Offset (none) -> 180
Connections:
- net +3.3V: now also U2.7 (VOUT)
- net DC: now also U2.4 (SHDN), U2.5 (VIN)
- net GND: now also U2.2 (GND)
- net at R5.2, R6.2: now also U2.3 (FB)
Changed lines of the file:
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@@
   (junction (at 124.46 33.655) (diameter 0) (color 0 0 0 0)
   )
+  (junction (at 135.89 42.545) (diameter 0) (color 0 0 0 0)
+  )
   (junction (at 50.8 43.18) (diameter 0) (color 0 0 0 0)
   )
@@
   )
   (junction (at 50.8 27.94) (diameter 0) (color 0 0 0 0)
-  )
-  (junction (at 135.89 42.545) (diameter 0) (color 0 0 0 0)
   )
   (junction (at 128.27 40.005) (diameter 0) (color 0 0 0 0)
@@
     (pin "2")
   )
+  (symbol (lib_id "RevK:LMR16006XDDCR") (at 135.89 32.385 0) (unit 1)
+    (in_bom yes) (on_board yes) (fields_autoplaced)
+    (property "Reference" "U2" (id 0) (at 153.67 27.5422 0))
+    (property "Value" "LMR16006XDDCR" (id 1) (at 153.67 30.0791 0))
+    (property "Footprint" "RevK:SOT-23-Thin-6-Reg" (id 2) (at 151.13 48.895 0)
+      (effects (font (size 1.27 1.27)) hide)
+    )
+    (property "Datasheet" "" (id 3) (at 147.32 29.845 0)
+      (effects (font (size 1.27 1.27)) hide)
+    )
+    (property "Manufacturer" "TI" (id 4) (at 163.83 46.99 0)
+      (effects (font (size 1.27 1.27)) hide)
+    )
+    (property "Part No" "LMR16006XDDCR" (id 5) (at 154.305 46.99 0)
+      (effects (font (size 1.27 1.27)) hide)
+    )
+    (property "LCSC Part #" "C87080" (id 6) (at 141.605 46.99 0)
+      (effects (font (size 1.27 1.27)) hide)
+    )
+    (property "JLCPCB Rotation Offset" "-90" (id 7) (at 166.37 46.99 0)
+      (effects (font (size 1.27 1.27)) hide)
+    )
+    (pin "1")
+    (pin "2")
+    (pin "3")
+    (pin "4")
+    (pin "5")
+    (pin "6")
+    (pin "7")
+  )
   (symbol (lib_id "power:GND") (at 142.24 83.82 270) (unit 1)
     (in_bom yes) (on_board yes) (fields_autoplaced)
@@
       (effects (font (size 1.27 1.27)) (justify right))
     )
-    (property "Footprint" "RevK:Hidden" (id 2) (at 151.765 34.29 0)
+    (property "Footprint" "RevK:C_0805_" (id 2) (at 151.765 34.29 0)
       (effects (font (size 1.27 1.27)) hide)
     )
@@
       (effects (font (size 1.27 1.27)) hide)
     )
-    (property "Note" "0603 or 0805" (id 4) (at 151.765 34.29 0)
-      (effects (font (size 1.27 1.27)) hide)
-    )
     (property "LCSC Part #" "C19110" (id 5) (at 151.765 34.29 0)
-      (effects (font (size 1.27 1.27)) hide)
-    )
-    (property "Part No" "" (id 6) (at 151.765 34.29 0)
       (effects (font (size 1.27 1.27)) hide)
     )
@@
       (effects (font (size 1.27 1.27)) (justify right))
     )
-    (property "Footprint" "RevK:Hidden" (id 2) (at 151.765 40.005 0)
+    (property "Footprint" "RevK:D_1206_" (id 2) (at 151.765 40.005 0)
       (effects (font (size 1.27 1.27)) hide)
     )
@@
     )
     (property "JLCPCB Rotation Offset" "180" (id 7) (at 151.765 40.005 0)
-      (effects (font (size 1.27 1.27)) hide)
-    )
-    (property "Part No" "" (id 7) (at 151.765 40.005 0)
-      (effects (font (size 1.27 1.27)) hide)
-    )
-    (property "Note" "" (id 8) (at 151.765 40.005 0)
       (effects (font (size 1.27 1.27)) hide)
     )
@@
     )
     (pin "1")
-  )
-  (symbol (lib_id "RevK:LMR16006+FB") (at 135.89 32.385 0) (unit 1)
-    (in_bom yes) (on_board yes) (fields_autoplaced)
-    (property "Reference" "U2" (id 0) (at 169.545 36.6303 0)
-      (effects (font (size 1.27 1.27)) (justify left))
-    )
-    (property "Value" "LMR16006XDDCR" (id 1) (at 169.545 39.1672 0)
-      (effects (font (size 1.27 1.27)) (justify left))
-    )
-    (property "Footprint" "RevK:SOT-23-Thin-6-Reg" (id 2) (at 147.32 29.845 0)
-      (effects (font (size 1.27 1.27)) hide)
-    )
-    (property "Datasheet" "~" (id 3) (at 147.32 29.845 0)
-      (effects (font (size 1.27 1.27)) hide)
-    )
-    (property "LCSC Part #" "C87080" (id 4) (at 135.89 32.385 0)
-      (effects (font (size 1.27 1.27)) hide)
-    )
-    (property "Manufacturer" "TI" (id 5) (at 135.89 32.385 0)
-      (effects (font (size 1.27 1.27)) hide)
-    )
-    (property "Part No" "LMR16006YQ3" (id 6) (at 135.89 32.385 0)
-      (effects (font (size 1.27 1.27)) hide)
-    )
-    (pin "1")
-    (pin "2")
-    (pin "3")
-    (pin "4")
-    (pin "5")
   )
   (symbol (lib_id "power:GND") (at 200.66 45.72 0) (unit 1)
@@
       (effects (font (size 1.27 1.27)) (justify right))
     )
-    (property "Footprint" "RevK:Hidden" (id 2) (at 151.765 36.195 0)
+    (property "Footprint" "RevK:C_0805_" (id 2) (at 151.765 36.195 0)
       (effects (font (size 1.27 1.27)) hide)
     )
@@
       (effects (font (size 1.27 1.27)) hide)
     )
-    (property "Note" "0603 or 0805" (id 4) (at 151.765 36.195 0)
-      (effects (font (size 1.27 1.27)) hide)
-    )
     (property "LCSC Part #" "C17024" (id 5) (at 151.765 36.195 0)
-      (effects (font (size 1.27 1.27)) hide)
-    )
-    (property "Part No" "" (id 6) (at 151.765 36.195 0)
       (effects (font (size 1.27 1.27)) hide)
     )
@@
       (effects (font (size 1.27 1.27)) (justify right))
     )
-    (property "Footprint" "RevK:Hidden" (id 2) (at 151.765 32.385 0)
+    (property "Footprint" "RevK:C_0603_" (id 2) (at 151.765 32.385 0)
       (effects (font (size 1.27 1.27)) hide)
     )
@@
     )
     (property "LCSC Part #" "C30926" (id 5) (at 151.765 32.385 0)
-      (effects (font (size 1.27 1.27)) hide)
-    )
-    (property "Part No" "" (id 6) (at 151.765 32.385 0)
       (effects (font (size 1.27 1.27)) hide)
     )
@@
       (effects (font (size 1.27 1.27)) (justify right))
     )
-    (property "Footprint" "RevK:Hidden" (id 2) (at 151.765 38.1 0)
+    (property "Footprint" "RevK:L_4x4_" (id 2) (at 151.765 38.1 0)
       (effects (font (size 1.27 1.27)) hide)
     )
@@
     )
     (property "LCSC Part #" "C354575" (id 6) (at 151.765 38.1 0)
-      (effects (font (size 1.27 1.27)) hide)
-    )
-    (property "Part No" "" (id 5) (at 151.765 38.1 0)
-      (effects (font (size 1.27 1.27)) hide)
-    )
-    (property "Note" "" (id 6) (at 151.765 38.1 0)
       (effects (font (size 1.27 1.27)) hide)
     )
@@
       (effects (font (size 1.27 1.27)) (justify left))
     )
-    (property "Footprint" "Package_TO_SOT_SMD:SOT-23" (id 2) (at 119.38 88.9 0)
+    (property "Footprint" "RevK:SOT-323_SC-70" (id 2) (at 119.38 88.9 0)
       (effects (font (size 1.27 1.27)) hide)
     )
@@
     )
     (property "LCSC Part #" "C504047" (id 5) (at 124.46 91.44 0)
+      (effects (font (size 1.27 1.27)) hide)
+    )
+    (property "JLCPCB Rotation Offset" "180" (id 6) (at 124.46 91.44 0)
       (effects (font (size 1.27 1.27)) hide)
     )
@@
     )
     (path "/b8671e87-1469-44e2-ab1b-2dbb18ba7eba"
-      (reference "C2") (unit 1) (value "100nF") (footprint "RevK:Hidden")
+      (reference "C2") (unit 1) (value "100nF") (footprint "RevK:C_0603_")
     )
     (path "/235f276c-84a0-4d76-963d-c6858a80fc70"
-      (reference "C3") (unit 1) (value "2.2uF") (footprint "RevK:Hidden")
+      (reference "C3") (unit 1) (value "2.2uF") (footprint "RevK:C_0805_")
     )
     (path "/9cc8d907-ad75-4ab2-9d9f-0dfdb290d4b7"
-      (reference "C4") (unit 1) (value "10uF") (footprint "RevK:Hidden")
+      (reference "C4") (unit 1) (value "10uF") (footprint "RevK:C_0805_")
     )
     (path "/296b967f-b7a9-453f-856a-7b874fdca3db"
@@
     )
     (path "/2a24d3f6-974c-420b-8ec3-07a5d48dea6b"
-      (reference "D2") (unit 1) (value "Schottky") (footprint "RevK:Hidden")
+      (reference "D2") (unit 1) (value "Schottky") (footprint "RevK:D_1206_")
     )
     (path "/af073fa6-a783-40f2-9751-692984a62ffc"
@@
     )
     (path "/bbd07ae0-123b-41d3-a93c-85b702312370"
-      (reference "L1") (unit 1) (value "6.8uH") (footprint "RevK:Hidden")
+      (reference "L1") (unit 1) (value "6.8uH") (footprint "RevK:L_4x4_")
     )
     (path "/ebcfdf36-110d-4f79-9de0-e4fcd76c1d6e"
-      (reference "Q3") (unit 1) (value "PMF250XNEX") (footprint "Package_TO_SOT_SMD:SOT-23")
+      (reference "Q3") (unit 1) (value "PMF250XNEX") (footprint "RevK:SOT-323_SC-70")
     )
     (path "/06b0f59d-5955-4cff-a86d-1a17e2ebba6e"
@@
       (reference "U1") (unit 1) (value "ESP32-PICO-MINI-02") (footprint "RevK:ESP32-PICO-MINI-02")
     )
-    (path "/56052c32-efab-47fa-b180-de209ff4cea9"
+    (path "/13e8e539-5f0a-494c-98f2-d0ff31f4eb09"
       (reference "U2") (unit 1) (value "LMR16006XDDCR") (footprint "RevK:SOT-23-Thin-6-Reg")
     )

Commit message: Tidy
Other:
- note removed: "Needs new LED from LCSC"
Changed lines of the file:
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@@
     (effects (font (size 1.27 1.27)) (justify left bottom))
-  )
-  (text "Needs new LED from LCSC" (at 99.695 143.51 0)
-    (effects (font (size 5 5)) (justify left bottom))
   )
   (global_label "G" (shape input) (at 81.28 63.5 0) (fields_autoplaced)

Commit message: Tidy
Parts:
- U2: value LMR16006XDDCR -> LMR16006YDDCR; JLCPCB Rotation Offset -90 -> 0; LCSC Part # C87080 -> C290195; Part No LMR16006XDDCR -> LMR16006YDDCR
Changed lines of the file:
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@@
     (in_bom yes) (on_board yes) (fields_autoplaced)
     (property "Reference" "U2" (id 0) (at 153.67 27.5422 0))
-    (property "Value" "LMR16006XDDCR" (id 1) (at 153.67 30.0791 0))
+    (property "Value" "LMR16006YDDCR" (id 1) (at 153.67 30.0791 0))
     (property "Footprint" "RevK:SOT-23-Thin-6-Reg" (id 2) (at 151.13 48.895 0)
       (effects (font (size 1.27 1.27)) hide)
@@
       (effects (font (size 1.27 1.27)) hide)
     )
-    (property "Part No" "LMR16006XDDCR" (id 5) (at 154.305 46.99 0)
-      (effects (font (size 1.27 1.27)) hide)
-    )
-    (property "LCSC Part #" "C87080" (id 6) (at 141.605 46.99 0)
-      (effects (font (size 1.27 1.27)) hide)
-    )
-    (property "JLCPCB Rotation Offset" "-90" (id 7) (at 166.37 46.99 0)
+    (property "Part No" "LMR16006YDDCR" (id 5) (at 154.305 46.99 0)
+      (effects (font (size 1.27 1.27)) hide)
+    )
+    (property "LCSC Part #" "C290195" (id 6) (at 141.605 46.99 0)
+      (effects (font (size 1.27 1.27)) hide)
+    )
+    (property "JLCPCB Rotation Offset" "0" (id 7) (at 166.37 46.99 0)
       (effects (font (size 1.27 1.27)) hide)
     )
@@
     )
     (path "/13e8e539-5f0a-494c-98f2-d0ff31f4eb09"
-      (reference "U2") (unit 1) (value "LMR16006XDDCR") (footprint "RevK:SOT-23-Thin-6-Reg")
-    )
-  )
+      (reference "U2") (unit 1) (value "LMR16006YDDCR") (footprint "RevK:SOT-23-Thin-6-Reg")
+    )
+  )
