File: PCB/Faikin3/Faikin.kicad_pcb (KiCad board)
At the start: 2 copper layers, 70 x 70 mm, 37 parts, among them J1 1x5, J2 Prog, Q3 PMF250XNEX, U1 ESP32-PICO-MINI-02, U2 Barcode, U3 MD8942, U4 Barcode

Commit message: Holes
Parts:
- moved H1 1.00 mm to (105.0, 40.0)
Changed lines of the file:
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@@
   )
   (footprint "MountingHole:MountingHole_2mm" (layer "F.Cu")
-    (at 106 40)
+    (at 105 40)
     (descr "Mounting Hole 2mm, no annular")
     (tags "mounting hole 2mm no annular")

Commit message: Re-panel
Parts:
- removed H1, H2, H3, H4: MountingHole, MountingHole:MountingHole_2mm
- removed U2: Barcode, RevK:EAN-5060634238151
- moved U4 46.0 mm to (153.5, 72.9)
- moved FID1 5.00 mm to (105.0, 32.9)
- moved FID2 5.00 mm to (165.0, 32.9)
- moved FID3 5.00 mm to (165.0, 97.2)
- moved FID4 5.00 mm to (105.0, 97.2)
- moved FID5 5.00 mm to (105.0, 32.9)
- moved FID6 5.00 mm to (165.0, 32.9)
- moved FID7 5.00 mm to (105.0, 97.2)
- moved FID8 5.00 mm to (165.0, 97.2)
- moved Q3 3.50 mm to (130.5, 61.4)
- moved R7 3.50 mm to (135.0, 61.9)
- moved C10 3.50 mm to (133.3, 56.3)
- moved C5 3.50 mm to (136.6, 53.4)
- moved C6 3.50 mm to (135.0, 60.1)
- moved C7 3.50 mm to (132.5, 60.2)
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Other:
- outline, holes or cut-outs redrawn
- board text added: "2 Designs, 0.8mm, Black, V-Cuts"

Commit message: Logo
Parts:
- added D1: BAV99S, RevK:SOT-363_SC-70-6, B.Cu at (137.0, 61.9)
- moved C1 3.13 mm to (140.1, 59.7)
- moved R4 1.12 mm to (138.3, 59.7), turned to 0 degrees
Routing:
- net +3.3V: track 39.1 -> 46.2 mm
- net RX: track 6.58 -> 11.2 mm, vias 1 -> 2
- net EN: track 9.45 -> 12.4 mm
- net DC: track 24.4 -> 26.8 mm
- net TX: track 4.92 -> 6.09 mm
- net GND: vias 4 -> 3

Commit message: (r)
Other:
- board text added: "®"
