File: PCB/Faikin3/Faikin.kicad_pcb (KiCad board)
At the start: 2 copper layers, 70 x 70 mm, 26 parts, among them J1 1x5, J2 Prog, Q3 PMF250XNEX, U1 ESP32-PICO-MINI-02, U3 MD8942, U4 Barcode

Commit message: VCUT
Parts:
- added V1: ~, RevK:VCUT70, F.Cu at (135.0, 51.0)
- added V2: ~, RevK:VCUT70, F.Cu at (135.0, 71.0)
Other:
- board text added: "${TITLE}"
- board text added: "RGB: 8/19/7"
- board text removed: "2 Designs, 0.8mm, Black"
- board text removed: "8/19/7"
- board text removed: "PCB-FAIKIN"

Commit message: test mask
Other:
- board text added: "060634"
- board text added: "OCR-B 1"
- board text added: "OCR-B 2"
- board text added: "OCR-B 3"
- board text added: "Ral 1"
- board text added: "Ral 1.2"
- board text added: "Ral 1.5"
- board text added: "Test mask"

Commit message: Test mask
Other:
- board text added: "Ral 2"

Commit message: Removed extra mask
Other:
- board text removed: "060634"
- board text removed: "OCR-B 1"
- board text removed: "OCR-B 2"
- board text removed: "OCR-B 3"
- board text removed: "Ral 1"
- board text removed: "Ral 1.2"
- board text removed: "Ral 1.5"
- board text removed: "Ral 2"
- board text removed: "Test mask"
