File: PCB/Faikin3/Faikin.kicad_sch (KiCad schematic)
At the start: 37 parts, among them J1 1x5, J2 Prog, Q3 PMF250XNEX, U1 ESP32-PICO-MINI-02, U2 Barcode, U3 MD8942, U4 Barcode

Commit message: tidy, new LED
Parts:
- removed D1: LED_BARG, RevK:MHS190RGBCT, symbol Device:LED_BARG
- removed R1: 300R, RevK:R_0402, symbol Device:R
- removed R2: 1K, RevK:R_0402, symbol Device:R
- removed R3: 100R, RevK:R_0402, symbol Device:R
- added D2: RGB, RevK:LED-RGB-1.6x1.6, symbol Device:LED_RBGA
- added R12: 220R, RevK:R_0402, symbol Device:R
- added R5: 680R, RevK:R_0402, symbol Device:R
- added R6: 2K, RevK:R_0402, symbol Device:R
Connections:
- net +3.3V: now also D2.4 (A)
- net B: now also R12.2
- net G: now also R6.2
- net R: now also R5.2
- new net: D2.2 (BK), R12.1
- new net: D2.1 (RK), R5.1
- new net: D2.3 (GK), R6.1

Commit message: Re-panel
Parts:
- removed H1, H2, H3, H4: MountingHole, MountingHole:MountingHole_2mm, symbol Mechanical:MountingHole
- removed U2: Barcode, RevK:EAN-5060634238151, symbol RevK:Barcode
Other:
- moved on the sheet: FID1, FID2, FID3, FID4, FID5, FID6, FID7, FID8

Commit message: Logo
Parts:
- added D1: BAV99S, RevK:SOT-363_SC-70-6, symbol Diode:BAV99S
Connections:
- net +3.3V: now also D1.2 (K2), D1.5 (K4)
- net GND: now also D1.1 (A1), D1.4 (A3)
- net RX: now also D1.3 (K1A2)
- net TX: now also D1.6 (K3A4)
Changed lines of the file:
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@@
+    )
+  )
+  (global_label "TX" (shape bidirectional) (at 118.11 132.715 270) (fields_autoplaced)
+    (effects (font (size 1.27 1.27)) (justify right))
+    (property "Intersheetrefs" "${INTERSHEET_REFS}" (at 118.11 138.0962 90)
+      (effects (font (size 1.27 1.27)) (justify right) hide)
     )
   )
@@
     )
   )
+  (global_label "RX" (shape bidirectional) (at 118.11 151.13 270) (fields_autoplaced)
+    (effects (font (size 1.27 1.27)) (justify right))
+    (property "Intersheetrefs" "${INTERSHEET_REFS}" (at 118.11 156.8136 90)
+      (effects (font (size 1.27 1.27)) (justify right) hide)
+    )
+  )
   (global_label "B" (shape input) (at 53.975 144.145 180) (fields_autoplaced)
     (effects (font (size 1.27 1.27)) (justify right))
@@
     )
   )
+  (symbol (lib_id "Diode:BAV99S") (at 118.11 146.05 0) (unit 2)
+    (in_bom yes) (on_board yes) (dnp no) (fields_autoplaced)
+    (property "Reference" "D1" (at 119.38 141.2 0)
+      (effects (font (size 1.27 1.27)))
+    )
+    (property "Value" "BAV99S" (at 119.38 143.248 0)
+      (effects (font (size 1.27 1.27)))
+    )
+    (property "Footprint" "RevK:SOT-363_SC-70-6" (at 118.11 158.75 0)
+      (effects (font (size 1.27 1.27)) hide)
+    )
+    (property "Datasheet" "https://assets.nexperia.com/documents/data-sheet/BAV99_SER.pdf" (at 118.11 146.05 0)
+      (effects (font (size 1.27 1.27)) hide)
+    )
+    (pin "1")
+    (pin "2")
+    (pin "6")
+    (pin "3")
+    (pin "4")
+    (pin "5")
+    (instances
+      (project "Faikin"
+        (path "/46c350bb-7de4-4e81-aafd-4af55e37aab0"
+          (reference "D1") (unit 2)
+        )
+      )
+    )
+  )
   (symbol (lib_id "Device:C") (at 143.51 95.25 180) (unit 1)
     (in_bom yes) (on_board yes) (dnp no)
@@
     )
   )
+  (symbol (lib_id "power:GND") (at 110.49 146.05 270) (unit 1)
+    (in_bom yes) (on_board yes) (dnp no) (fields_autoplaced)
+    (property "Reference" "#PWR05" (at 104.14 146.05 0)
+      (effects (font (size 1.27 1.27)) hide)
+    )
+    (property "Value" "GND" (at 107.3151 146.05 90)
+      (effects (font (size 1.27 1.27)) (justify right))
+    )
+    (property "Footprint" "" (at 110.49 146.05 0)
+      (effects (font (size 1.27 1.27)) hide)
+    )
+    (property "Datasheet" "" (at 110.49 146.05 0)
+      (effects (font (size 1.27 1.27)) hide)
+    )
+    (pin "1")
+    (instances
+      (project "Faikin"
+        (path "/46c350bb-7de4-4e81-aafd-4af55e37aab0"
+          (reference "#PWR05") (unit 1)
+        )
+      )
+    )
+  )
   (symbol (lib_id "Mechanical:Fiducial") (at 259.08 161.925 0) (unit 1)
     (in_bom no) (on_board yes) (dnp no) (fields_autoplaced)
@@
         (path "/46c350bb-7de4-4e81-aafd-4af55e37aab0"
           (reference "FID8") (unit 1)
+        )
+      )
+    )
+  )
+  (symbol (lib_id "power:+3.3V") (at 125.73 146.05 270) (unit 1)
+    (in_bom yes) (on_board yes) (dnp no)
+    (property "Reference" "#PWR07" (at 121.92 146.05 0)
+      (effects (font (size 1.27 1.27)) hide)
+    )
+    (property "Value" "+3.3V" (at 128.9812 146.431 90)
+      (effects (font (size 1.27 1.27)) (justify left))
+    )
+    (property "Footprint" "" (at 125.73 146.05 0)
+      (effects (font (size 1.27 1.27)) hide)
+    )
+    (property "Datasheet" "" (at 125.73 146.05 0)
+      (effects (font (size 1.27 1.27)) hide)
+    )
+    (pin "1")
+    (instances
+      (project "Faikin"
+        (path "/46c350bb-7de4-4e81-aafd-4af55e37aab0"
+          (reference "#PWR07") (unit 1)
+        )
+      )
+      (project "Reference"
+        (path "/825c70b0-4860-42b7-97dc-86bfa46e06fd"
+          (reference "#PWR04") (unit 1)
         )
       )
@@
     )
   )
+  (symbol (lib_id "power:GND") (at 110.49 127.635 270) (unit 1)
+    (in_bom yes) (on_board yes) (dnp no) (fields_autoplaced)
+    (property "Reference" "#PWR04" (at 104.14 127.635 0)
+      (effects (font (size 1.27 1.27)) hide)
+    )
+    (property "Value" "GND" (at 107.3151 127.635 90)
+      (effects (font (size 1.27 1.27)) (justify right))
+    )
+    (property "Footprint" "" (at 110.49 127.635 0)
+      (effects (font (size 1.27 1.27)) hide)
+    )
+    (property "Datasheet" "" (at 110.49 127.635 0)
+      (effects (font (size 1.27 1.27)) hide)
+    )
+    (pin "1")
+    (instances
+      (project "Faikin"
+        (path "/46c350bb-7de4-4e81-aafd-4af55e37aab0"
+          (reference "#PWR04") (unit 1)
+        )
+      )
+    )
+  )
   (symbol (lib_id "power:GND") (at 233.68 41.275 0) (unit 1)
     (in_bom yes) (on_board yes) (dnp no)
@@
         )
       )
+    )
+  )
+  (symbol (lib_id "Diode:BAV99S") (at 118.11 127.635 0) (unit 1)
+    (in_bom yes) (on_board yes) (dnp no) (fields_autoplaced)
+    (property "Reference" "D1" (at 119.38 122.785 0)
+      (effects (font (size 1.27 1.27)))
+    )
+    (property "Value" "BAV99S" (at 119.38 124.833 0)
+      (effects (font (size 1.27 1.27)))
+    )
+    (property "Footprint" "RevK:SOT-363_SC-70-6" (at 118.11 140.335 0)
+      (effects (font (size 1.27 1.27)) hide)
+    )
+    (property "Datasheet" "https://assets.nexperia.com/documents/data-sheet/BAV99_SER.pdf" (at 118.11 127.635 0)
+      (effects (font (size 1.27 1.27)) hide)
+    )
+    (pin "1")
+    (pin "2")
+    (pin "6")
+    (pin "3")
+    (pin "4")
+    (pin "5")
+    (instances
+      (project "Faikin"
+        (path "/46c350bb-7de4-4e81-aafd-4af55e37aab0"
+          (reference "D1") (unit 1)
+        )
+      )
+    )
+  )
+  (symbol (lib_id "power:+3.3V") (at 125.73 127.635 270) (unit 1)
+    (in_bom yes) (on_board yes) (dnp no)
+    (property "Reference" "#PWR06" (at 121.92 127.635 0)
+      (effects (font (size 1.27 1.27)) hide)
+    )
+    (property "Value" "+3.3V" (at 128.9812 128.016 90)
+      (effects (font (size 1.27 1.27)) (justify left))
+    )
+    (property "Footprint" "" (at 125.73 127.635 0)
+      (effects (font (size 1.27 1.27)) hide)
+    )
+    (property "Datasheet" "" (at 125.73 127.635 0)
+      (effects (font (size 1.27 1.27)) hide)
+    )
+    (pin "1")
+    (instances
+      (project "Faikin"
+        (path "/46c350bb-7de4-4e81-aafd-4af55e37aab0"
+          (reference "#PWR06") (unit 1)
+        )
+      )
+      (project "Reference"
+        (path "/825c70b0-4860-42b7-97dc-86bfa46e06fd"
+          (reference "#PWR04") (unit 1)
+        )
+      )

Commit message: BAV99S part fix
Parts:
- D1: JLCPCB Rotation Offset (none) -> 90; LCSC Part # (none) -> C712378
Changed lines of the file:
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@@
+      (effects (font (size 1.27 1.27)) hide)
+    )
+    (property "LCSC Part #" "C712378" (at 118.11 146.05 0)
+      (effects (font (size 1.27 1.27)) hide)
+    )
+    (property "JLCPCB Rotation Offset" "90" (at 118.11 146.05 0)
       (effects (font (size 1.27 1.27)) hide)
     )
@@
       (effects (font (size 1.27 1.27)) hide)
     )
+    (property "LCSC Part #" "C712378" (at 118.11 127.635 0)
+      (effects (font (size 1.27 1.27)) hide)
+    )
+    (property "JLCPCB Rotation Offset" "90" (at 118.11 127.635 0)
+      (effects (font (size 1.27 1.27)) hide)
+    )

Commit message: V Cuts
Other:
- moved on the sheet: C10, C8, C9, L2, R10, R11, R9, U3

Commit message: Better rails
Parts:
- removed FID1, FID2, FID3, FID4, FID5, FID6, FID7, FID8: Fiducial, Fiducial:Fiducial_1mm_Mask2mm, symbol Mechanical:Fiducial
- added PCB1: 70x70, RevK:PCB7070, symbol RevK:PCB
Changed lines of the file:
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@@
-    )
-  )
-  (symbol (lib_id "Mechanical:Fiducial") (at 259.08 151.765 0) (unit 1)
-    (in_bom no) (on_board yes) (dnp no) (fields_autoplaced)
-    (property "Reference" "FID6" (at 261.239 150.741 0)
-      (effects (font (size 1.27 1.27)) (justify left))
-    )
-    (property "Value" "Fiducial" (at 261.239 152.789 0)
-      (effects (font (size 1.27 1.27)) (justify left))
-    )
-    (property "Footprint" "Fiducial:Fiducial_1mm_Mask2mm" (at 259.08 151.765 0)
-      (effects (font (size 1.27 1.27)) hide)
-    )
-    (property "Datasheet" "~" (at 259.08 151.765 0)
-      (effects (font (size 1.27 1.27)) hide)
-    )
-    (instances
-      (project "Faikin"
-        (path "/46c350bb-7de4-4e81-aafd-4af55e37aab0"
-          (reference "FID6") (unit 1)
-        )
-      )
     )
   )
@@
     )
   )
-  (symbol (lib_id "Mechanical:Fiducial") (at 271.145 151.765 0) (unit 1)
-    (in_bom no) (on_board yes) (dnp no) (fields_autoplaced)
-    (property "Reference" "FID2" (at 273.304 150.741 0)
-      (effects (font (size 1.27 1.27)) (justify left))
-    )
-    (property "Value" "Fiducial" (at 273.304 152.789 0)
-      (effects (font (size 1.27 1.27)) (justify left))
-    )
-    (property "Footprint" "Fiducial:Fiducial_1mm_Mask2mm" (at 271.145 151.765 0)
-      (effects (font (size 1.27 1.27)) hide)
-    )
-    (property "Datasheet" "~" (at 271.145 151.765 0)
-      (effects (font (size 1.27 1.27)) hide)
-    )
-    (instances
-      (project "Faikin"
-        (path "/46c350bb-7de4-4e81-aafd-4af55e37aab0"
-          (reference "FID2") (unit 1)
-        )
-      )
-    )
-  )
-  (symbol (lib_id "Mechanical:Fiducial") (at 259.08 156.845 0) (unit 1)
-    (in_bom no) (on_board yes) (dnp no) (fields_autoplaced)
-    (property "Reference" "FID7" (at 261.239 155.821 0)
-      (effects (font (size 1.27 1.27)) (justify left))
-    )
-    (property "Value" "Fiducial" (at 261.239 157.869 0)
-      (effects (font (size 1.27 1.27)) (justify left))
-    )
-    (property "Footprint" "Fiducial:Fiducial_1mm_Mask2mm" (at 259.08 156.845 0)
-      (effects (font (size 1.27 1.27)) hide)
-    )
-    (property "Datasheet" "~" (at 259.08 156.845 0)
-      (effects (font (size 1.27 1.27)) hide)
-    )
-    (instances
-      (project "Faikin"
-        (path "/46c350bb-7de4-4e81-aafd-4af55e37aab0"
-          (reference "FID7") (unit 1)
-        )
-      )
-    )
-  )
-  (symbol (lib_id "Mechanical:Fiducial") (at 259.08 146.685 0) (unit 1)
-    (in_bom no) (on_board yes) (dnp no) (fields_autoplaced)
-    (property "Reference" "FID5" (at 261.239 145.661 0)
-      (effects (font (size 1.27 1.27)) (justify left))
-    )
-    (property "Value" "Fiducial" (at 261.239 147.709 0)
-      (effects (font (size 1.27 1.27)) (justify left))
-    )
-    (property "Footprint" "Fiducial:Fiducial_1mm_Mask2mm" (at 259.08 146.685 0)
-      (effects (font (size 1.27 1.27)) hide)
-    )
-    (property "Datasheet" "~" (at 259.08 146.685 0)
-      (effects (font (size 1.27 1.27)) hide)
-    )
-    (instances
-      (project "Faikin"
-        (path "/46c350bb-7de4-4e81-aafd-4af55e37aab0"
-          (reference "FID5") (unit 1)
-        )
-      )
-    )
-  )
   (symbol (lib_id "Device:C") (at 143.51 85.09 0) (unit 1)
     (in_bom yes) (on_board yes) (dnp no)
@@
         (path "/46c350bb-7de4-4e81-aafd-4af55e37aab0"
           (reference "#PWR05") (unit 1)
-        )
-      )
-    )
-  )
-  (symbol (lib_id "Mechanical:Fiducial") (at 259.08 161.925 0) (unit 1)
-    (in_bom no) (on_board yes) (dnp no) (fields_autoplaced)
-    (property "Reference" "FID8" (at 261.239 160.901 0)
-      (effects (font (size 1.27 1.27)) (justify left))
-    )
-    (property "Value" "Fiducial" (at 261.239 162.949 0)
-      (effects (font (size 1.27 1.27)) (justify left))
-    )
-    (property "Footprint" "Fiducial:Fiducial_1mm_Mask2mm" (at 259.08 161.925 0)
-      (effects (font (size 1.27 1.27)) hide)
-    )
-    (property "Datasheet" "~" (at 259.08 161.925 0)
-      (effects (font (size 1.27 1.27)) hide)
-    )
-    (instances
-      (project "Faikin"
-        (path "/46c350bb-7de4-4e81-aafd-4af55e37aab0"
-          (reference "FID8") (unit 1)
         )
       )
@@
     )
   )
-  (symbol (lib_id "Mechanical:Fiducial") (at 271.145 156.845 0) (unit 1)
-    (in_bom no) (on_board yes) (dnp no) (fields_autoplaced)
-    (property "Reference" "FID3" (at 273.304 155.821 0)
-      (effects (font (size 1.27 1.27)) (justify left))
-    )
-    (property "Value" "Fiducial" (at 273.304 157.869 0)
-      (effects (font (size 1.27 1.27)) (justify left))
-    )
-    (property "Footprint" "Fiducial:Fiducial_1mm_Mask2mm" (at 271.145 156.845 0)
-      (effects (font (size 1.27 1.27)) hide)
-    )
-    (property "Datasheet" "~" (at 271.145 156.845 0)
-      (effects (font (size 1.27 1.27)) hide)
-    )
-    (instances
-      (project "Faikin"
-        (path "/46c350bb-7de4-4e81-aafd-4af55e37aab0"
-          (reference "FID3") (unit 1)
-        )
-      )
-    )
-  )
   (symbol (lib_id "power:GND") (at 100.33 31.75 0) (unit 1)
     (in_bom yes) (on_board yes) (dnp no) (fields_autoplaced)
@@
         (path "/46c350bb-7de4-4e81-aafd-4af55e37aab0"
           (reference "#PWR0110") (unit 1)
+        )
+      )
+    )
+  )
+  (symbol (lib_id "RevK:PCB") (at 262.255 174.625 0) (unit 1)
+    (in_bom no) (on_board yes) (dnp no)
+    (property "Reference" "PCB1" (at 262.255 184.785 0)
+      (effects (font (size 1.27 1.27)) hide)
+    )
+    (property "Value" "70x70" (at 262.255 174.625 0)
+      (effects (font (size 1.27 1.27)))
+    )
+    (property "Footprint" "RevK:PCB7070" (at 262.255 168.91 0)
+      (effects (font (size 1.27 1.27)) hide)
+    )
+    (property "Datasheet" "" (at 262.255 174.625 0)
+      (effects (font (size 1.27 1.27)) hide)
+    )
+    (instances
+      (project "Faikin"
+        (path "/46c350bb-7de4-4e81-aafd-4af55e37aab0"
+          (reference "PCB1") (unit 1)
         )
       )
@@
     )
   )
-  (symbol (lib_id "Mechanical:Fiducial") (at 271.145 161.925 0) (unit 1)
-    (in_bom no) (on_board yes) (dnp no) (fields_autoplaced)
-    (property "Reference" "FID4" (at 273.304 160.901 0)
-      (effects (font (size 1.27 1.27)) (justify left))
-    )
-    (property "Value" "Fiducial" (at 273.304 162.949 0)
-      (effects (font (size 1.27 1.27)) (justify left))
-    )
-    (property "Footprint" "Fiducial:Fiducial_1mm_Mask2mm" (at 271.145 161.925 0)
-      (effects (font (size 1.27 1.27)) hide)
-    )
-    (property "Datasheet" "~" (at 271.145 161.925 0)
-      (effects (font (size 1.27 1.27)) hide)
-    )
-    (instances
-      (project "Faikin"
-        (path "/46c350bb-7de4-4e81-aafd-4af55e37aab0"
-          (reference "FID4") (unit 1)
-        )
-      )
-    )
-  )
   (symbol (lib_id "Device:C") (at 39.37 27.94 90) (unit 1)
     (in_bom yes) (on_board yes) (dnp no) (fields_autoplaced)
@@
         )
       )
-    )
-  )
-  (symbol (lib_id "Mechanical:Fiducial") (at 271.145 146.685 0) (unit 1)
-    (in_bom no) (on_board yes) (dnp no) (fields_autoplaced)
-    (property "Reference" "FID1" (at 273.304 145.661 0)
-      (effects (font (size 1.27 1.27)) (justify left))
-    )
-    (property "Value" "Fiducial" (at 273.304 147.709 0)
-      (effects (font (size 1.27 1.27)) (justify left))
-    )
-    (property "Footprint" "Fiducial:Fiducial_1mm_Mask2mm" (at 271.145 146.685 0)
-      (effects (font (size 1.27 1.27)) hide)
-    )
-    (property "Datasheet" "~" (at 271.145 146.685 0)
-      (effects (font (size 1.27 1.27)) hide)
-    )
-    (instances
-      (project "Faikin"
-        (path "/46c350bb-7de4-4e81-aafd-4af55e37aab0"
-          (reference "FID1") (unit 1)
-        )
-      )

Commit message: VCUT
Parts:
- added V1, V2: ~, RevK:VCUT70, symbol RevK:VCUT
Changed lines of the file:
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@@
+    )
+  )
+  (symbol (lib_id "RevK:VCUT") (at 262.255 177.8 0) (unit 1)
+    (in_bom yes) (on_board yes) (dnp no) (fields_autoplaced)
+    (property "Reference" "V2" (at 262.255 176.53 0)
+      (effects (font (size 1.27 1.27)) hide)
+    )
+    (property "Value" "~" (at 262.255 177.8 0)
+      (effects (font (size 1.27 1.27)))
+    )
+    (property "Footprint" "RevK:VCUT70" (at 262.255 179.07 0)
+      (effects (font (size 1.27 1.27)) hide)
+    )
+    (property "Datasheet" "" (at 262.255 177.8 0)
+      (effects (font (size 1.27 1.27)) hide)
+    )
+    (instances
+      (project "Faikin"
+        (path "/46c350bb-7de4-4e81-aafd-4af55e37aab0"
+          (reference "V2") (unit 1)
+        )
+      )
     )
   )
@@
         )
       )
+    )
+  )
+  (symbol (lib_id "RevK:VCUT") (at 262.255 171.45 0) (unit 1)
+    (in_bom yes) (on_board yes) (dnp no) (fields_autoplaced)
+    (property "Reference" "V1" (at 262.255 170.18 0)
+      (effects (font (size 1.27 1.27)) hide)
+    )
+    (property "Value" "~" (at 262.255 171.45 0)
+      (effects (font (size 1.27 1.27)))
+    )
+    (property "Footprint" "RevK:VCUT70" (at 262.255 172.72 0)
+      (effects (font (size 1.27 1.27)) hide)
+    )
+    (property "Datasheet" "" (at 262.255 171.45 0)
+      (effects (font (size 1.27 1.27)) hide)
+    )
+    (instances
+      (project "Faikin"
+        (path "/46c350bb-7de4-4e81-aafd-4af55e37aab0"
+          (reference "V1") (unit 1)
+        )
+      )

Commit message: test mask
Parts:
- V1, V2: now left out of the parts list
Changed lines of the file:
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@@
   )
   (symbol (lib_id "RevK:VCUT") (at 262.255 177.8 0) (unit 1)
-    (in_bom yes) (on_board yes) (dnp no) (fields_autoplaced)
+    (in_bom no) (on_board yes) (dnp no) (fields_autoplaced)
     (property "Reference" "V2" (at 262.255 176.53 0)
       (effects (font (size 1.27 1.27)) hide)
@@
     )
     (property "Datasheet" "" (at 262.255 177.8 0)
+      (effects (font (size 1.27 1.27)) hide)
+    )
+    (property "Sim.Enable" "0" (at 262.255 177.8 0)
       (effects (font (size 1.27 1.27)) hide)
     )
@@
   )
   (symbol (lib_id "RevK:VCUT") (at 262.255 171.45 0) (unit 1)
-    (in_bom yes) (on_board yes) (dnp no) (fields_autoplaced)
+    (in_bom no) (on_board yes) (dnp no) (fields_autoplaced)
     (property "Reference" "V1" (at 262.255 170.18 0)
       (effects (font (size 1.27 1.27)) hide)
@@
       (effects (font (size 1.27 1.27)) hide)
     )
+    (property "Sim.Enable" "0" (at 262.255 171.45 0)
+      (effects (font (size 1.27 1.27)) hide)
+    )
