File: PCB/Faikin2/Faikin.kicad_sch (KiCad schematic)
At the start: 30 parts, among them J1 1x5, J2 Shelly, Q1 BSS138PS, U2 Barcode, U2 ESP32-S3-MINI-1, U3 MD8942

Commit message: Smaller
Connections:
- no-connect marks 32 -> 31
Other:
- moved on the sheet: C3, R1
Changed lines of the file:
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@@
   (junction (at 79.375 58.42) (diameter 0) (color 0 0 0 0)
   )
+  (junction (at 85.725 102.235) (diameter 0) (color 0 0 0 0)
+  )
   (junction (at 139.7 75.565) (diameter 0) (color 0 0 0 0)
   )
@@
   )
   (junction (at 143.51 91.44) (diameter 0) (color 0 0 0 0)
-  )
-  (junction (at 85.725 102.87) (diameter 0) (color 0 0 0 0)
   )
   (junction (at 143.51 88.9) (diameter 0) (color 0 0 0 0)
@@
   (no_connect (at 79.375 81.28))
   (no_connect (at 79.375 73.66))
-  (no_connect (at 48.895 102.87))
   (no_connect (at 48.895 73.66))
   (wire (pts (xy 135.255 91.44) (xy 143.51 91.44))
@@
     (stroke (width 0) (type default))
   )
-  (wire (pts (xy 79.375 102.87) (xy 85.725 102.87))
+  (wire (pts (xy 79.375 102.235) (xy 85.725 102.235))
     (stroke (width 0) (type default))
   )
@@
     )
   )
-  (symbol (lib_id "power:+3.3V") (at 85.725 95.25 0) (unit 1)
-    (in_bom yes) (on_board yes) (dnp no) (fields_autoplaced)
-    (property "Reference" "#PWR0106" (at 85.725 99.06 0)
-      (effects (font (size 1.27 1.27)) hide)
-    )
-    (property "Value" "+3.3V" (at 85.725 91.6742 0)
-      (effects (font (size 1.27 1.27)))
-    )
-    (property "Footprint" "" (at 85.725 95.25 0)
-      (effects (font (size 1.27 1.27)) hide)
-    )
-    (property "Datasheet" "" (at 85.725 95.25 0)
+  (symbol (lib_id "power:+3.3V") (at 85.725 94.615 0) (unit 1)
+    (in_bom yes) (on_board yes) (dnp no) (fields_autoplaced)
+    (property "Reference" "#PWR0106" (at 85.725 98.425 0)
+      (effects (font (size 1.27 1.27)) hide)
+    )
+    (property "Value" "+3.3V" (at 85.725 91.0392 0)
+      (effects (font (size 1.27 1.27)))
+    )
+    (property "Footprint" "" (at 85.725 94.615 0)
+      (effects (font (size 1.27 1.27)) hide)
+    )
+    (property "Datasheet" "" (at 85.725 94.615 0)
       (effects (font (size 1.27 1.27)) hide)
     )
@@
     )
   )
-  (symbol (lib_id "power:GND") (at 85.725 110.49 0) (unit 1)
-    (in_bom yes) (on_board yes) (dnp no) (fields_autoplaced)
-    (property "Reference" "#PWR0105" (at 85.725 116.84 0)
-      (effects (font (size 1.27 1.27)) hide)
-    )
-    (property "Value" "GND" (at 85.725 114.9334 0)
-      (effects (font (size 1.27 1.27)))
-    )
-    (property "Footprint" "" (at 85.725 110.49 0)
-      (effects (font (size 1.27 1.27)) hide)
-    )
-    (property "Datasheet" "" (at 85.725 110.49 0)
+  (symbol (lib_id "power:GND") (at 85.725 109.855 0) (unit 1)
+    (in_bom yes) (on_board yes) (dnp no) (fields_autoplaced)
+    (property "Reference" "#PWR0105" (at 85.725 116.205 0)
+      (effects (font (size 1.27 1.27)) hide)
+    )
+    (property "Value" "GND" (at 85.725 114.2984 0)
+      (effects (font (size 1.27 1.27)))
+    )
+    (property "Footprint" "" (at 85.725 109.855 0)
+      (effects (font (size 1.27 1.27)) hide)
+    )
+    (property "Datasheet" "" (at 85.725 109.855 0)
       (effects (font (size 1.27 1.27)) hide)
     )
@@
     )
   )
-  (symbol (lib_id "Device:C") (at 85.725 106.68 0) (unit 1)
-    (in_bom yes) (on_board yes) (dnp no) (fields_autoplaced)
-    (property "Reference" "C3" (at 88.646 105.8453 0)
-      (effects (font (size 1.27 1.27)) (justify left))
-    )
-    (property "Value" "1uF" (at 88.646 108.3822 0)
-      (effects (font (size 1.27 1.27)) (justify left))
-    )
-    (property "Footprint" "RevK:C_0402" (at 86.6902 110.49 0)
-      (effects (font (size 1.27 1.27)) hide)
-    )
-    (property "Datasheet" "~" (at 85.725 106.68 0)
+  (symbol (lib_id "Device:C") (at 85.725 106.045 0) (unit 1)
+    (in_bom yes) (on_board yes) (dnp no) (fields_autoplaced)
+    (property "Reference" "C3" (at 88.646 105.2103 0)
+      (effects (font (size 1.27 1.27)) (justify left))
+    )
+    (property "Value" "1uF" (at 88.646 107.7472 0)
+      (effects (font (size 1.27 1.27)) (justify left))
+    )
+    (property "Footprint" "RevK:C_0402" (at 86.6902 109.855 0)
+      (effects (font (size 1.27 1.27)) hide)
+    )
+    (property "Datasheet" "~" (at 85.725 106.045 0)
       (effects (font (size 1.27 1.27)) hide)
     )
@@
     )
   )
-  (symbol (lib_id "Device:R") (at 85.725 99.06 0) (unit 1)
-    (in_bom yes) (on_board yes) (dnp no)
-    (property "Reference" "R1" (at 87.63 99.06 90)
-      (effects (font (size 1.27 1.27)))
-    )
-    (property "Value" "10K" (at 85.725 99.06 90)
-      (effects (font (size 1.27 1.27)))
-    )
-    (property "Footprint" "RevK:R_0402" (at 83.947 99.06 90)
-      (effects (font (size 1.27 1.27)) hide)
-    )
-    (property "Datasheet" "~" (at 85.725 99.06 0)
-      (effects (font (size 1.27 1.27)) hide)
-    )
+  (symbol (lib_id "Device:R") (at 85.725 98.425 0) (unit 1)
+    (in_bom yes) (on_board yes) (dnp no)
+    (property "Reference" "R1" (at 87.63 98.425 90)
+      (effects (font (size 1.27 1.27)))
+    )
+    (property "Value" "10K" (at 85.725 98.425 90)
+      (effects (font (size 1.27 1.27)))
+    )
+    (property "Footprint" "RevK:R_0402" (at 83.947 98.425 90)
+      (effects (font (size 1.27 1.27)) hide)
+    )
+    (property "Datasheet" "~" (at 85.725 98.425 0)
+      (effects (font (size 1.27 1.27)) hide)
+    )

Commit message: SMaller
Changed lines of the file:
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@@
     )
     (property "Value" "AJK" (at 250.825 174.625 0)
-      (effects (font (size 1.27 1.27)) (justify left))
+      (effects (font (size 1.27 1.27)) (justify left) hide)
     )
     (property "Footprint" "RevK:AJK" (at 250.19 177.165 0)
