File: PCB/Faikin2/Faikin.kicad_sch (KiCad schematic)
At the start: 31 parts, among them J1 1x5, J2 Shelly, J3 USB-PROG, Q1 BSS138PS, U2 ESP32-S3-MINI-1, U3 MD8942

Commit message: Wider still
Changed lines of the file:
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@@
     )
   )
-  (symbol (lib_id "RevK:VCUT") (at 262.255 172.085 0) (unit 1)
+  (symbol (lib_id "RevK:VCUT") (at 262.255 171.45 0) (unit 1)
     (in_bom no) (on_board yes) (dnp no) (fields_autoplaced)
-    (property "Reference" "V3" (at 262.255 170.815 0)
-      (effects (font (size 1.27 1.27)) hide)
-    )
-    (property "Value" "~" (at 262.255 172.085 0)
-      (effects (font (size 1.27 1.27)))
-    )
-    (property "Footprint" "RevK:VCUT70" (at 262.255 173.355 0)
-      (effects (font (size 1.27 1.27)) hide)
-    )
-    (property "Datasheet" "" (at 262.255 172.085 0)
-      (effects (font (size 1.27 1.27)) hide)
-    )
-    (property "Sim.Enable" "0" (at 262.255 172.085 0)
+    (property "Reference" "V3" (at 262.255 170.18 0)
+      (effects (font (size 1.27 1.27)) hide)
+    )
+    (property "Value" "~" (at 262.255 171.45 0)
+      (effects (font (size 1.27 1.27)))
+    )
+    (property "Footprint" "RevK:VCUT70" (at 262.255 172.72 0)
+      (effects (font (size 1.27 1.27)) hide)
+    )
+    (property "Datasheet" "" (at 262.255 171.45 0)
+      (effects (font (size 1.27 1.27)) hide)
+    )
+    (property "Sim.Enable" "0" (at 262.255 171.45 0)
       (effects (font (size 1.27 1.27)) hide)
     )
@@
     )
   )
-  (symbol (lib_id "RevK:VCUT") (at 262.255 177.165 0) (unit 1)
+  (symbol (lib_id "RevK:VCUT") (at 262.255 177.8 0) (unit 1)
     (in_bom no) (on_board yes) (dnp no) (fields_autoplaced)
-    (property "Reference" "V4" (at 262.255 175.895 0)
-      (effects (font (size 1.27 1.27)) hide)
-    )
-    (property "Value" "~" (at 262.255 177.165 0)
-      (effects (font (size 1.27 1.27)))
-    )
-    (property "Footprint" "RevK:VCUT70" (at 262.255 178.435 0)
-      (effects (font (size 1.27 1.27)) hide)
-    )
-    (property "Datasheet" "" (at 262.255 177.165 0)
-      (effects (font (size 1.27 1.27)) hide)
-    )
-    (property "Sim.Enable" "0" (at 262.255 177.165 0)
+    (property "Reference" "V4" (at 262.255 176.53 0)
+      (effects (font (size 1.27 1.27)) hide)
+    )
+    (property "Value" "~" (at 262.255 177.8 0)
+      (effects (font (size 1.27 1.27)))
+    )
+    (property "Footprint" "RevK:VCUT70" (at 262.255 179.07 0)
+      (effects (font (size 1.27 1.27)) hide)
+    )
+    (property "Datasheet" "" (at 262.255 177.8 0)
+      (effects (font (size 1.27 1.27)) hide)
+    )
+    (property "Sim.Enable" "0" (at 262.255 177.8 0)
       (effects (font (size 1.27 1.27)) hide)
     )
@@
     )
   )
-  (symbol (lib_id "RevK:VCUT") (at 262.255 177.8 0) (unit 1)
+  (symbol (lib_id "RevK:VCUT") (at 262.255 177.165 0) (unit 1)
     (in_bom no) (on_board yes) (dnp no) (fields_autoplaced)
-    (property "Reference" "V2" (at 262.255 176.53 0)
-      (effects (font (size 1.27 1.27)) hide)
-    )
-    (property "Value" "~" (at 262.255 177.8 0)
-      (effects (font (size 1.27 1.27)))
-    )
-    (property "Footprint" "RevK:VCUT70" (at 262.255 179.07 0)
-      (effects (font (size 1.27 1.27)) hide)
-    )
-    (property "Datasheet" "" (at 262.255 177.8 0)
-      (effects (font (size 1.27 1.27)) hide)
-    )
-    (property "Sim.Enable" "0" (at 262.255 177.8 0)
+    (property "Reference" "V2" (at 262.255 175.895 0)
+      (effects (font (size 1.27 1.27)) hide)
+    )
+    (property "Value" "~" (at 262.255 177.165 0)
+      (effects (font (size 1.27 1.27)))
+    )
+    (property "Footprint" "RevK:VCUT70" (at 262.255 178.435 0)
+      (effects (font (size 1.27 1.27)) hide)
+    )
+    (property "Datasheet" "" (at 262.255 177.165 0)
+      (effects (font (size 1.27 1.27)) hide)
+    )
+    (property "Sim.Enable" "0" (at 262.255 177.165 0)
       (effects (font (size 1.27 1.27)) hide)
     )
@@
     )
   )
-  (symbol (lib_name "Hidden_1") (lib_id "RevK:Hidden") (at 259.08 173.99 0) (unit 1)
+  (symbol (lib_name "Hidden_1") (lib_id "RevK:Hidden") (at 259.08 173.355 0) (unit 1)
     (in_bom no) (on_board yes) (dnp no) (fields_autoplaced)
-    (property "Reference" "Z2" (at 260.4262 173.99 0)
+    (property "Reference" "Z2" (at 260.4262 173.355 0)
       (effects (font (size 1.27 1.27)) (justify left) hide)
     )
-    (property "Value" "Hidden" (at 260.4262 175.2021 0)
+    (property "Value" "Hidden" (at 260.4262 174.5671 0)
       (effects (font (size 1.27 1.27)) (justify left) hide)
     )
-    (property "Footprint" "RevK:PCB-Join1" (at 259.08 172.085 0)
-      (effects (font (size 1.27 1.27)) hide)
-    )
-    (property "Datasheet" "" (at 259.08 173.99 0)
-      (effects (font (size 1.27 1.27)) hide)
-    )
-    (property "Part No" "" (at 259.08 173.99 0)
-      (effects (font (size 1.27 1.27)) hide)
-    )
-    (property "Note" "" (at 259.08 173.99 0)
+    (property "Footprint" "RevK:PCB-Join1" (at 259.08 171.45 0)
+      (effects (font (size 1.27 1.27)) hide)
+    )
+    (property "Datasheet" "" (at 259.08 173.355 0)
+      (effects (font (size 1.27 1.27)) hide)
+    )
+    (property "Part No" "" (at 259.08 173.355 0)
+      (effects (font (size 1.27 1.27)) hide)
+    )
+    (property "Note" "" (at 259.08 173.355 0)
       (effects (font (size 1.27 1.27)) hide)
     )
@@
     )
   )
-  (symbol (lib_id "RevK:VCUT") (at 262.255 171.45 0) (unit 1)
+  (symbol (lib_id "RevK:VCUT") (at 262.255 172.085 0) (unit 1)
     (in_bom no) (on_board yes) (dnp no) (fields_autoplaced)
-    (property "Reference" "V1" (at 262.255 170.18 0)
-      (effects (font (size 1.27 1.27)) hide)
-    )
-    (property "Value" "~" (at 262.255 171.45 0)
-      (effects (font (size 1.27 1.27)))
-    )
-    (property "Footprint" "RevK:VCUT70" (at 262.255 172.72 0)
-      (effects (font (size 1.27 1.27)) hide)
-    )
-    (property "Datasheet" "" (at 262.255 171.45 0)
-      (effects (font (size 1.27 1.27)) hide)
-    )
-    (property "Sim.Enable" "0" (at 262.255 171.45 0)
+    (property "Reference" "V1" (at 262.255 170.815 0)
+      (effects (font (size 1.27 1.27)) hide)
+    )
+    (property "Value" "~" (at 262.255 172.085 0)
+      (effects (font (size 1.27 1.27)))
+    )
+    (property "Footprint" "RevK:VCUT70" (at 262.255 173.355 0)
+      (effects (font (size 1.27 1.27)) hide)
+    )
+    (property "Datasheet" "" (at 262.255 172.085 0)
+      (effects (font (size 1.27 1.27)) hide)
+    )
+    (property "Sim.Enable" "0" (at 262.255 172.085 0)
       (effects (font (size 1.27 1.27)) hide)
     )
@@
     )
   )
-  (symbol (lib_name "Hidden_1") (lib_id "RevK:Hidden") (at 265.43 173.99 0) (unit 1)
+  (symbol (lib_name "Hidden_1") (lib_id "RevK:Hidden") (at 265.43 173.355 0) (unit 1)
     (in_bom no) (on_board yes) (dnp no) (fields_autoplaced)
-    (property "Reference" "Z3" (at 266.7762 173.99 0)
+    (property "Reference" "Z3" (at 266.7762 173.355 0)
       (effects (font (size 1.27 1.27)) (justify left) hide)
     )
-    (property "Value" "Hidden" (at 266.7762 175.2021 0)
+    (property "Value" "Hidden" (at 266.7762 174.5671 0)
       (effects (font (size 1.27 1.27)) (justify left) hide)
     )
-    (property "Footprint" "RevK:PCB-Join1" (at 265.43 172.085 0)
-      (effects (font (size 1.27 1.27)) hide)
-    )
-    (property "Datasheet" "" (at 265.43 173.99 0)
-      (effects (font (size 1.27 1.27)) hide)
-    )
-    (property "Part No" "" (at 265.43 173.99 0)
-      (effects (font (size 1.27 1.27)) hide)
-    )
-    (property "Note" "" (at 265.43 173.99 0)
-      (effects (font (size 1.27 1.27)) hide)
-    )
+    (property "Footprint" "RevK:PCB-Join1" (at 265.43 171.45 0)
+      (effects (font (size 1.27 1.27)) hide)
+    )
+    (property "Datasheet" "" (at 265.43 173.355 0)
+      (effects (font (size 1.27 1.27)) hide)
+    )
+    (property "Part No" "" (at 265.43 173.355 0)
+      (effects (font (size 1.27 1.27)) hide)
+    )
+    (property "Note" "" (at 265.43 173.355 0)
+      (effects (font (size 1.27 1.27)) hide)
+    )

Commit message: Library update
Other:
- note added: "Careful routing of Rx line to avoid the regulator"
Changed lines of the file:
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@@
     (stroke (width 0) (type default))
   )
-  (text "A cap to GND seems obvious\nBut experiments show it\nmakes it way more noisy!"
-    (at 129.54 107.95 0)
+  (text "Careful routing of Rx line\nto avoid the regulator" (at 140.97 101.6 0)
     (effects (font (size 1.27 1.27)) (justify left bottom))
   )
+  (text "A cap to GND seems obvious\nBut experiments show it\nmakes it way more noisy!"
+    (at 146.05 73.66 0)
+    (effects (font (size 1.27 1.27)) (justify left bottom))
+  )
