File: PCB/Faikin2/Faikin.kicad_pcb (KiCad board)
At the start: 2 copper layers, 70 x 70 mm, 30 parts, among them J1 1x5, J3 Shelly, Q1 BSS138PS, U2 Barcode, U3 MD8942, U4 ESP32-S3-MINI-1

Commit message: Silkscreen
Parts:
- moved Logo1 0.63 mm to (136.1, 62.9)

Commit message: Tidy
Parts:
- J3: moved to B.Cu
Routing:
- net Net-(Q1B-SP): track 9.81 -> 8.59 mm, vias 2 -> 0

Commit message: SMaller
Parts:
- removed Logo1: AJK, RevK:AJK
- moved J3 14.8 mm to (133.8, 61.0)
- moved C2 9.19 mm to (138.5, 59.0), turned to 180 degrees
- moved R11 6.81 mm to (142.5, 66.9), turned to -90 degrees
- moved R9 6.73 mm to (140.0, 68.0), turned to 0 degrees
- moved R10 5.71 mm to (137.5, 66.9), turned to -90 degrees
- moved C8 4.99 mm to (142.5, 64.8), turned to 90 degrees
- moved U3 4.09 mm to (140.0, 66.1), turned to 180 degrees
- moved R1 3.72 mm to (143.5, 62.5), turned to 180 degrees
- moved C5 3.64 mm to (141.5, 59.0), turned to 0 degrees
- moved C9 3.33 mm to (137.5, 64.8), turned to -90 degrees
- moved C6 3.00 mm to (137.9, 54.0)
- moved D2 3.00 mm to (139.7, 55.9)
- moved R12 3.00 mm to (137.9, 55.0)
- moved R3 3.00 mm to (140.3, 54.0)
- moved R5 3.00 mm to (137.9, 55.9)
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Routing:
- net Net-(J3-0): track 41.0 -> 14.0 mm
- net Net-(J3-Rx): track 41.9 -> 19.8 mm
- net +3.3V: track 65.9 -> 44.3 mm, vias 2 -> 3
- net Net-(J3-Tx): track 36.3 -> 21.1 mm
- net Net-(Q1B-SP): track 8.59 -> 17.7 mm, vias 0 -> 2
- net DC: track 9.45 -> 12.3 mm, vias 1 -> 0
- net Net-(Q1A-GN): track 5.15 -> 6.76 mm
- net Net-(J1-Pin_1): track 11.5 -> 12.7 mm, vias 1 -> 0
- net GND: track 1.20 -> 2.20 mm, vias 11 -> 14
- net TX: track 7.33 -> 6.33 mm
- net Net-(J1-Pin_3): track 2.00 -> 1.10 mm
- net Net-(J1-Pin_2): track 2.00 -> 1.10 mm
Other:
- board text added: "A"
- board text added: "RGB: 34/33/48"
- board text removed: "21"
- board text removed: "34/33/48"
- board text removed: "47"

Commit message: Prettier tracks
Parts:
- moved C5 1.15 mm to (140.3, 59.0)
- moved C4 0.50 mm to (143.5, 58.5)
- moved R8 0.50 mm to (143.5, 59.5)
Routing:
- net Net-(J3-Rx): track 19.8 -> 17.8 mm
- net Net-(J1-Pin_3): track 1.10 -> 2.83 mm
- net Net-(Q1B-SP): track 17.7 -> 16.2 mm
- net +3.3V: track 44.3 -> 45.5 mm
- net Net-(J1-Pin_2): track 1.10 -> 1.94 mm
- net GND: vias 14 -> 15

Commit message: 45mm x 36mm break outs to replace in-situ
Parts:
- added V3: ~, RevK:VCUT70, F.Cu at (152.1, 65.0)
- added V4: ~, RevK:VCUT70, F.Cu at (107.1, 65.0)
- added V5: ~, RevK:VCUT70, F.Cu at (135.0, 43.0)
- added V6: ~, RevK:VCUT70, F.Cu at (135.0, 79.0)

Commit message: Adjusted for panel and barcode
Parts:
- moved R10 6.00 mm to (137.5, 60.9)
- moved R11 6.00 mm to (142.5, 60.9)
- moved C2 6.00 mm to (138.5, 53.0)
- moved C3 6.00 mm to (143.5, 54.5)
- moved C4 6.00 mm to (143.5, 52.5)
- moved C5 6.00 mm to (140.3, 53.0)
- moved C6 6.00 mm to (137.9, 48.0)
- moved C8 6.00 mm to (142.5, 58.8)
- moved C9 6.00 mm to (137.5, 58.8)
- moved D2 6.00 mm to (139.7, 49.9)
- moved J1 6.00 mm to (145.6, 50.0)
- moved J3 6.00 mm to (133.8, 55.0)
- moved L2 6.00 mm to (140.0, 55.5)
- moved Q1 6.00 mm to (142.0, 50.0)
- moved R1 6.00 mm to (143.5, 56.5)
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
Commit message: USB-PROG
Parts:
- removed J3: Shelly, RevK:Shelly
- added J2: USB_A, RevK:USB-PROG, B.Cu at (133.8, 55.0)
- turned V5 to 180 degrees
Connections:
- U4 pad 23: unconnected-(U4-GPIO19-Pad23) -> Net-(J2-D-)
- U4 pad 24: unconnected-(U4-GPIO20-Pad24) -> Net-(J2-D+)
- U4 pad 39: Net-(J3-Tx) -> unconnected-(U4-GPIO43-Pad39)
- U4 pad 4: Net-(J3-0) -> unconnected-(U4-GPIO0-Pad4)
- U4 pad 40: Net-(J3-Rx) -> unconnected-(U4-GPIO44-Pad40)
Routing:
- net Net-(J3-Tx): track 21.3 -> 0.00 mm, vias 1 -> 0
- net Net-(J3-Rx): track 17.8 -> 0.00 mm, vias 1 -> 0
- net Net-(J3-0): track 13.7 -> 0.00 mm, vias 1 -> 0
- net DC: track 12.0 -> 24.6 mm
- net +3.3V: track 45.5 -> 33.4 mm
- net Net-(J2-D-): track 0.00 -> 4.17 mm
- net Net-(J2-D+): track 0.00 -> 2.87 mm
- net GND: vias 15 -> 17
Other:
- board text added: "21"
- board text added: "47"
- board text removed: "26"
- board text removed: "27"
