File: PCB/Faikin/Faikin.kicad_sch (KiCad schematic)
At the start: 28 parts, among them J1 1x5, J2 Shelly, J3 USB-PROG, Q1 BSS138PS, U2 ESP32-S3-MINI-1, U3 MD8942

Commit message: Tidy, for order
Changed lines of the file:
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@@
     )
   )
-  (symbol (lib_id "RevK:ES05D1MC10") (at 132.08 107.315 270) (unit 1)
-    (in_bom yes) (on_board yes) (dnp no) (fields_autoplaced)
-    (property "Reference" "D3" (at 134.112 107.315 90)
-      (effects (font (size 1.27 1.27)) (justify left))
-    )
-    (property "Value" "~" (at 132.08 107.315 0)
-      (effects (font (size 1.27 1.27)))
-    )
-    (property "Footprint" "RevK:DFN1006-2L" (at 135.255 107.95 0)
-      (effects (font (size 1.27 1.27)) hide)
-    )
-    (property "Datasheet" "" (at 132.08 107.315 0)
-      (effects (font (size 1.27 1.27)) hide)
-    )
-    (property "LCSC Part #" "C5137770" (at 128.905 107.315 0)
+  (symbol (lib_id "RevK:ES05D1MC10") (at 132.08 104.775 270) (unit 1)
+    (in_bom yes) (on_board yes) (dnp no) (fields_autoplaced)
+    (property "Reference" "D3" (at 134.112 104.775 90)
+      (effects (font (size 1.27 1.27)) (justify left))
+    )
+    (property "Value" "~" (at 132.08 104.775 0)
+      (effects (font (size 1.27 1.27)))
+    )
+    (property "Footprint" "RevK:DFN1006-2L" (at 135.255 105.41 0)
+      (effects (font (size 1.27 1.27)) hide)
+    )
+    (property "Datasheet" "" (at 132.08 104.775 0)
+      (effects (font (size 1.27 1.27)) hide)
+    )
+    (property "LCSC Part #" "C5137770" (at 128.905 104.775 0)
       (effects (font (size 1.27 1.27)) hide)
     )
@@
     )
   )
-  (symbol (lib_id "RevK:ES05D1MC10") (at 132.08 81.915 270) (unit 1)
-    (in_bom yes) (on_board yes) (dnp no) (fields_autoplaced)
-    (property "Reference" "D2" (at 134.112 81.915 90)
-      (effects (font (size 1.27 1.27)) (justify left))
-    )
-    (property "Value" "~" (at 132.08 81.915 0)
-      (effects (font (size 1.27 1.27)))
-    )
-    (property "Footprint" "RevK:DFN1006-2L" (at 135.255 82.55 0)
-      (effects (font (size 1.27 1.27)) hide)
-    )
-    (property "Datasheet" "" (at 132.08 81.915 0)
-      (effects (font (size 1.27 1.27)) hide)
-    )
-    (property "LCSC Part #" "C5137770" (at 128.905 81.915 0)
+  (symbol (lib_id "RevK:ES05D1MC10") (at 132.08 79.375 270) (unit 1)
+    (in_bom yes) (on_board yes) (dnp no) (fields_autoplaced)
+    (property "Reference" "D2" (at 134.112 79.375 90)
+      (effects (font (size 1.27 1.27)) (justify left))
+    )
+    (property "Value" "~" (at 132.08 79.375 0)
+      (effects (font (size 1.27 1.27)))
+    )
+    (property "Footprint" "RevK:DFN1006-2L" (at 135.255 80.01 0)
+      (effects (font (size 1.27 1.27)) hide)
+    )
+    (property "Datasheet" "" (at 132.08 79.375 0)
+      (effects (font (size 1.27 1.27)) hide)
+    )
+    (property "LCSC Part #" "C5137770" (at 128.905 79.375 0)
       (effects (font (size 1.27 1.27)) hide)
     )
@@
     )
   )
-  (symbol (lib_id "power:GND") (at 132.08 113.665 0) (unit 1)
-    (in_bom yes) (on_board yes) (dnp no) (fields_autoplaced)
-    (property "Reference" "#PWR024" (at 132.08 120.015 0)
-      (effects (font (size 1.27 1.27)) hide)
-    )
-    (property "Value" "GND" (at 132.08 117.2408 0)
-      (effects (font (size 1.27 1.27)))
-    )
-    (property "Footprint" "" (at 132.08 113.665 0)
-      (effects (font (size 1.27 1.27)) hide)
-    )
-    (property "Datasheet" "" (at 132.08 113.665 0)
+  (symbol (lib_id "power:GND") (at 132.08 108.585 0) (unit 1)
+    (in_bom yes) (on_board yes) (dnp no) (fields_autoplaced)
+    (property "Reference" "#PWR024" (at 132.08 114.935 0)
+      (effects (font (size 1.27 1.27)) hide)
+    )
+    (property "Value" "GND" (at 132.08 112.1608 0)
+      (effects (font (size 1.27 1.27)))
+    )
+    (property "Footprint" "" (at 132.08 108.585 0)
+      (effects (font (size 1.27 1.27)) hide)
+    )
+    (property "Datasheet" "" (at 132.08 108.585 0)
       (effects (font (size 1.27 1.27)) hide)
     )
@@
     )
   )
-  (symbol (lib_id "power:GND") (at 132.08 88.265 0) (unit 1)
-    (in_bom yes) (on_board yes) (dnp no) (fields_autoplaced)
-    (property "Reference" "#PWR03" (at 132.08 94.615 0)
-      (effects (font (size 1.27 1.27)) hide)
-    )
-    (property "Value" "GND" (at 132.08 91.8408 0)
-      (effects (font (size 1.27 1.27)))
-    )
-    (property "Footprint" "" (at 132.08 88.265 0)
-      (effects (font (size 1.27 1.27)) hide)
-    )
-    (property "Datasheet" "" (at 132.08 88.265 0)
-      (effects (font (size 1.27 1.27)) hide)
-    )
+  (symbol (lib_id "power:GND") (at 132.08 83.185 0) (unit 1)
+    (in_bom yes) (on_board yes) (dnp no) (fields_autoplaced)
+    (property "Reference" "#PWR03" (at 132.08 89.535 0)
+      (effects (font (size 1.27 1.27)) hide)
+    )
+    (property "Value" "GND" (at 132.08 86.7608 0)
+      (effects (font (size 1.27 1.27)))
+    )
+    (property "Footprint" "" (at 132.08 83.185 0)
+      (effects (font (size 1.27 1.27)) hide)
+    )
+    (property "Datasheet" "" (at 132.08 83.185 0)
+      (effects (font (size 1.27 1.27)) hide)
+    )

Commit message: Tidy BOM
Parts:
- J3: now left out of the parts list
Changed lines of the file:
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@@
   )
   (symbol (lib_id "RevK:USB-PROG") (at 107.315 137.16 0) (unit 1)
-    (in_bom yes) (on_board yes) (dnp no) (fields_autoplaced)
+    (in_bom no) (on_board yes) (dnp no) (fields_autoplaced)
     (property "Reference" "J3" (at 107.315 125.3957 0)
       (effects (font (size 1.27 1.27)))

Commit message: Library update
Parts:
- C8: value 10uF 50V -> 10uF 35V; LCSC Part # C1591 -> C194427
Changed lines of the file:
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@@
       (effects (font (size 1.27 1.27)) (justify left))
     )
-    (property "Value" "10uF 50V" (at 157.48 45.085 0)
+    (property "Value" "10uF 35V" (at 157.48 45.085 0)
       (effects (font (size 1.27 1.27)) (justify left))
     )
@@
       (effects (font (size 1.27 1.27)) hide)
     )
-    (property "LCSC Part #" "C1591" (at 151.13 45.085 0)
+    (property "LCSC Part #" "C194427" (at 151.13 45.085 0)
       (effects (font (size 1.27 1.27)) hide)
     )
