File: PCB/Faikin+/Faikin+.kicad_pcb (KiCad board)
At the start: 2 copper layers, 70 x 70 mm, 30 parts, among them J1 1x5, J2 Shelly, J3 USB-PROG, J4 1x5, Q1 BSS138PS, Q2 BSS138PS, U3 MD8942, U4 ESP32-S3-MINI-1

Commit message: New pass through
Parts:
- added C1: 100nF, RevK:C_0402, F.Cu at (145.7, 48.8)
- added C3: 100nF, RevK:C_0402, F.Cu at (145.7, 79.2)
- moved D1 4.12 mm to (148.0, 78.0)
- moved D4 4.12 mm to (148.0, 50.0)
- moved R2 2.00 mm to (144.0, 50.0)
- moved D2 1.00 mm to (144.0, 78.0), turned to 0 degrees
- moved R1 1.00 mm to (144.0, 77.0), turned to 0 degrees
- turned Q1 to 90 degrees
- turned Q2 to -90 degrees
Connections:
- U4 pad 16: GND -> unconnected-(U4-GPIO12-Pad16)
- U4 pad 17: GND -> unconnected-(U4-GPIO13-Pad17)
- U4 pad 18: GND -> unconnected-(U4-GPIO14-Pad18)
- U4 pad 19: GND -> unconnected-(U4-GPIO15-Pad19)
- U4 pad 20: GND -> unconnected-(U4-GPIO16-Pad20)
- U4 pad 21: GND -> unconnected-(U4-GPIO17-Pad21)
- U4 pad 22: GND -> unconnected-(U4-GPIO18-Pad22)
Routing:
- net +3.3V: track 14.6 -> 60.8 mm, vias 0 -> 1
- net DC: track 22.5 -> 51.5 mm, vias 0 -> 1
- net Net-(D1-O): track 0.00 -> 28.8 mm
- net GND: track 3.35 -> 28.5 mm, vias 0 -> 28
- net LED: track 0.00 -> 23.4 mm, vias 0 -> 2
- net RX: track 0.00 -> 18.7 mm, vias 0 -> 2
- net TX: track 0.00 -> 18.4 mm, vias 0 -> 2
- net S21TX: track 46.3 -> 58.3 mm
- net TX2: track 0.00 -> 5.45 mm
- net RX2: track 0.00 -> 5.28 mm
- net Net-(U4-EN): track 16.9 -> 19.5 mm, vias 0 -> 2
- net Net-(J1-Pin_1): track 58.2 -> 56.3 mm
- net S21RX: track 69.1 -> 69.8 mm
Other:
- board text added: "35"
- board text added: "36"
