File: PCB/Faikin+/Faikin+.kicad_sch (KiCad schematic)
At the start: 30 parts, among them J1 1x5, J2 Shelly, J3 USB-PROG, J4 1x5, Q1 BSS138PS, Q2 BSS138PS, U2 ESP32-S3-MINI-1, U3 MD8942

Commit message: New pass through
Parts:
- added C1, C3: 100nF, RevK:C_0402, symbol Device:C
Connections:
- net +3.3V: now also C1.1, C3.1
- net GND: now also C1.2, C3.2; no longer U2.16 (GPIO12), U2.17 (GPIO13), U2.18 (GPIO14), U2.19 (GPIO15), U2.20 (GPIO16), U2.21 (GPIO17), U2.22 (GPIO18)
- no-connect marks 23 -> 30
Other:
- moved on the sheet: D1

Commit message: Tweaks
Parts:
- R9: LCSC Part # (none) -> C138062
Changed lines of the file:
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@@
       (effects (font (size 1.27 1.27)) hide)
     )
-    (property "Part No" "" (at 151.13 50.8 0)
+    (property "LCSC Part #" "C138062" (at 151.13 50.8 0)
       (effects (font (size 1.27 1.27)) hide)
     )
-    (property "Note" "" (at 151.13 50.8 0)
-      (effects (font (size 1.27 1.27)) hide)
-    )
