File: PCB/Faikin+/Faikin+.kicad_sch (KiCad schematic)
At the start: 32 parts, among them J1 1x5, J2 Shelly, J3 USB-PROG, J4 1x5, Q1 BSS138PS, Q2 BSS138PS, U2 ESP32-S3-MINI-1, U3 MD8942

Commit message: New header
Parts:
- removed J2: Shelly, RevK:Shelly, symbol RevK:Shelly
- removed J3: USB-PROG, RevK:USB-PROG, symbol RevK:USB-PROG
- added J5: TC2030-USB-NL-DS, RevK:Tag-Connect_TC2030-IDC-NL_2x03_P1.27mm_Vertical, symbol RevK:TC2030-USB-NL
Connections:
- net D+: now also J5.4 (D+)
- net D-: now also J5.3 (D-)
- net DC: now also J5.1 (VBUS), J5.2 (VBUS)
- net GND: now also J5.5 (GND), J5.6 (GND)
- no-connect marks 30 -> 34
